File: RLOOP_BMS_V2/Clock Generator.sch (KiCad schematic (older format))
At the start: 6 parts, among them IC1 FXO-HC736R-1.000, IC2 SN74AUP1G74DCUR

Commit message: Footprint work
starting to assign footprints to parts
Parts:
- C1, C2: footprint (none) -> Capacitors_SMD:C_0603
- IC1: footprint (none) -> rLoop_Footprints:Oscillator_SMD_FOX_HC3_4pin_7.0x5.0mm
- R1, R2: footprint (none) -> Resistors_SMD:R_0603
Changed lines of the file:
@@
 F 0 "IC1" H 3800 4400 60  0000 C CNN
 F 1 "FXO-HC736R-1.000" H 4200 4300 60  0000 C CNN
-F 2 "" H 3500 4000 60  0001 C CNN
+F 2 "rLoop_Footprints:Oscillator_SMD_FOX_HC3_4pin_7.0x5.0mm" H 3500 4000 60  0001 C CNN
 F 3 "" H 3500 4000 60  0001 C CNN
 	1    3500 4000
@@
 F 0 "R2" V 4250 3900 50  0000 C CNN
 F 1 "47R / .1W / 1% / SMD 0603" V 4450 4400 50  0000 C CNN
-F 2 "" V 4280 3900 50  0001 C CNN
+F 2 "Resistors_SMD:R_0603" V 4280 3900 50  0001 C CNN
 F 3 "" H 4350 3900 50  0001 C CNN
 	1    4350 3900
@@
 F 0 "R1" V 6500 5500 50  0000 C CNN
 F 1 "47R / .1 W / 1% / SMD 0603" V 6700 5450 50  0000 C CNN
-F 2 "" V 6530 5500 50  0001 C CNN
+F 2 "Resistors_SMD:R_0603" V 6530 5500 50  0001 C CNN
 F 3 "" H 6600 5500 50  0001 C CNN
 	1    6600 5500
@@
 F 0 "C1" V 3200 3450 50  0000 L CNN
 F 1 "100n / 50V / 10% / SMD 0603" V 3450 2200 50  0000 L CNN
-F 2 "" H 3388 3400 50  0001 C CNN
+F 2 "Capacitors_SMD:C_0603" H 3388 3400 50  0001 C CNN
 F 3 "" H 3350 3550 50  0001 C CNN
 	1    3350 3550
@@
 F 0 "C2" V 6500 3500 50  0000 L CNN
 F 1 "100n / 50V / 10% / SMD 0603" V 6600 3500 50  0000 L CNN
-F 2 "" H 6788 3400 50  0001 C CNN
+F 2 "Capacitors_SMD:C_0603" H 6788 3400 50  0001 C CNN
 F 3 "" H 6750 3550 50  0001 C CNN
 	1    6750 3550

Commit message: footprint and layout work WIP
Parts:
- IC2: footprint (none) -> rLoop_Footprints:TI_sn74aup1g74_UQFN-0.6mm
Changed lines of the file:
@@
 F 0 "IC2" H 6200 4650 60  0000 C CNN
 F 1 "SN74AUP1G74DCUR" H 6000 4550 60  0000 C CNN
-F 2 "" H 6600 4100 60  0001 C CNN
+F 2 "rLoop_Footprints:TI_sn74aup1g74_UQFN-0.6mm" H 6600 4100 60  0001 C CNN
 F 3 "" H 6600 4100 60  0001 C CNN
 	1    6600 4100
