File: RLOOP_BMS_V2/rLoop BMS v2.kicad_pcb (KiCad board)
At the start: 2 copper layers, 186 parts, among them IC1 FXO-HC736R-1.000, IC2 SN74AUP1G74DCUR, IC3 ATA6870N-PLQW-1, IC4 ATA6870N-PLQW-1, IC5 ATA6870N-PLQW-1, J1 CONN_02X07, J2 2-1586041-0, Q1 FDN337N, Q10 PMV20ENR, Q11 PMV20ENR, Q12 PMV20ENR, Q13 PMV20ENR, Q14 PMV20ENR, Q15 PMV20ENR, Q16 PMV20ENR, Q17 PMV20ENR, Q18 PMV20ENR, Q19 PMV20ENR, Q2 PMV20ENR, Q3 PMV20ENR, Q4 PMV20ENR, Q5 PMV20ENR, Q6 PMV20ENR, Q7 PMV20ENR, Q8 PMV20ENR, Q9 PMV20ENR, U1 VOS618A-2X001T

Commit message: board layout wip
Parts:
- C3, C4: footprint Capacitors_SMD:C_0603 -> Capacitors_SMD:C_1206
- J2: value 2-1586041-0 -> 2-640387-0; footprint rLoop_Footprints:TE_2-1586041-0-2x10 -> rLoop_Footprints:TE_2-640387-0
- moved IC2 244.1 mm to (291.5, 15.0), turned to 90 degrees
- moved C25 241.7 mm to (302.5, 16.5), turned to 90 degrees
- moved C26 238.7 mm to (302.5, 8.50), turned to 90 degrees
- moved C36 232.3 mm to (302.5, 121.5), turned to 90 degrees
- moved C35 231.2 mm to (302.5, 127.0), turned to 90 degrees
- moved C24 230.0 mm to (302.5, 23.5), turned to 90 degrees
- moved C37 229.5 mm to (302.5, 113.5), turned to 90 degrees
- moved C34 228.8 mm to (305.5, 131.5)
- moved C38 227.2 mm to (302.5, 107.0), turned to 90 degrees
- moved C39 223.7 mm to (302.5, 99.0), turned to 90 degrees
- moved C23 223.1 mm to (302.5, 31.5), turned to 90 degrees
- moved C12 221.1 mm to (302.5, 61.5), turned to 90 degrees
- moved U1 211.2 mm to (273.5, 118.5), turned to 270 degrees
- moved C21 210.3 mm to (302.5, 46.0), turned to 90 degrees
- moved IC4 209.1 mm to (291.0, 28.5), turned to 180 degrees
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Connections:
- J2 pad 1: GND_1 -> Net-(J2-Pad1)
- J2 pad 10: /DISCHARGE Top/CELL_9 -> /DISCHARGE Top/CELL_10
- J2 pad 11: /DISCHARGE Top/CELL_10 -> /DISCHARGE Top/CELL_9
- J2 pad 12: /DISCHARGE Top/CELL_11 -> /DISCHARGE Top/CELL_8
- J2 pad 13: /DISCHARGE Top/CELL_12 -> /DISCHARGE Top/CELL_7
- J2 pad 14: /DISCHARGE Top/CELL_13 -> /DISCHARGE Top/CELL_6
- J2 pad 15: /DISCHARGE Top/CELL_14 -> /DISCHARGE Top/CELL_5
- J2 pad 16: /DISCHARGE Top/CELL_15 -> /DISCHARGE Top/CELL_4
- J2 pad 17: /DISCHARGE Top/CELL_16 -> /DISCHARGE Top/CELL_3
- J2 pad 18: /DISCHARGE Top/CELL_16 -> /DISCHARGE Top/CELL_2
- J2 pad 19: /DISCHARGE Top/CELL_18 -> /DISCHARGE Top/CELL_1
- J2 pad 2: /DISCHARGE Top/CELL_1 -> /DISCHARGE Top/CELL_18
- J2 pad 20: Net-(J2-Pad20) -> GND_1
- J2 pad 3: /DISCHARGE Top/CELL_2 -> /DISCHARGE Top/CELL_16
- J2 pad 4: /DISCHARGE Top/CELL_3 -> /DISCHARGE Top/CELL_16
- J2 pad 5: /DISCHARGE Top/CELL_4 -> /DISCHARGE Top/CELL_15
- J2 pad 6: /DISCHARGE Top/CELL_5 -> /DISCHARGE Top/CELL_14
- J2 pad 7: /DISCHARGE Top/CELL_6 -> /DISCHARGE Top/CELL_13
- J2 pad 8: /DISCHARGE Top/CELL_7 -> /DISCHARGE Top/CELL_12
- J2 pad 9: /DISCHARGE Top/CELL_8 -> /DISCHARGE Top/CELL_11
Other:
- board outline added: 129.2 x 133.8 mm

Commit message: PCB Layout WIP
Parts:
- added REF**: Heatsink, rLoop_Footprints:Heatsink_TO-220_542502B00000G, F.Cu at (333.0, 39.0)
- added REF**: Heatsink, rLoop_Footprints:Heatsink_TO-220_542502B00000G, F.Cu at (333.0, 4.00)
- added REF**: Heatsink, rLoop_Footprints:Heatsink_TO-220_542502B00000G, F.Cu at (333.0, 11.0)
- added REF**: Heatsink, rLoop_Footprints:Heatsink_TO-220_542502B00000G, F.Cu at (333.0, 18.0)
- added REF**: Heatsink, rLoop_Footprints:Heatsink_TO-220_542502B00000G, F.Cu at (333.0, 102.5)
- added REF**: Heatsink, rLoop_Footprints:Heatsink_TO-220_542502B00000G, F.Cu at (333.0, 109.5)
- added REF**: Heatsink, rLoop_Footprints:Heatsink_TO-220_542502B00000G, F.Cu at (333.0, 88.5)
- added REF**: Heatsink, rLoop_Footprints:Heatsink_TO-220_542502B00000G, F.Cu at (333.0, 95.5)
- added REF**: Heatsink, rLoop_Footprints:Heatsink_TO-220_542502B00000G, F.Cu at (333.0, 116.5)
- added REF**: Heatsink, rLoop_Footprints:Heatsink_TO-220_542502B00000G, F.Cu at (333.0, 123.5)
- added REF**: Heatsink, rLoop_Footprints:Heatsink_TO-220_542502B00000G, F.Cu at (333.0, 46.0)
- added REF**: Heatsink, rLoop_Footprints:Heatsink_TO-220_542502B00000G, F.Cu at (333.0, 74.5)
- added REF**: Heatsink, rLoop_Footprints:Heatsink_TO-220_542502B00000G, F.Cu at (333.0, 53.0)
- added REF**: Heatsink, rLoop_Footprints:Heatsink_TO-220_542502B00000G, F.Cu at (333.0, 60.0)
- added REF**: Heatsink, rLoop_Footprints:Heatsink_TO-220_542502B00000G, F.Cu at (333.0, 67.0)
- added REF**: Heatsink, rLoop_Footprints:Heatsink_TO-220_542502B00000G, F.Cu at (333.0, 81.5)
- added REF**: Heatsink, rLoop_Footprints:Heatsink_TO-220_542502B00000G, F.Cu at (333.0, 32.0)
- added REF**: Heatsink, rLoop_Footprints:Heatsink_TO-220_542502B00000G, F.Cu at (333.0, 25.0)
- R39, R40, R41, R42, R43, R44, R64, R65, R66, R67, R68, R69, R89, R90, R91, R92, R93, R94: footprint TO_SOT_Packages_THT:TO-220-2_Vertical -> rLoop_Footprints:Res_MP930
- moved R35 23.1 mm to (335.0, 104.5)
- moved R33 22.9 mm to (334.5, 118.5)
- moved R34 22.8 mm to (334.5, 111.5)
- moved R85 22.6 mm to (335.5, 20.0), turned to 180 degrees
- moved R59 22.6 mm to (335.0, 69.0)
- moved R86 22.5 mm to (335.5, 13.0)
- moved R88 22.5 mm to (335.0, -1.00)
- moved R36 22.5 mm to (334.5, 97.5)
- moved R60 22.5 mm to (335.0, 62.0), turned to 180 degrees
- moved R61 22.5 mm to (335.0, 55.0), turned to 180 degrees
- moved R37 22.3 mm to (334.5, 90.5)
- moved R38 22.3 mm to (334.5, 83.5)
- moved R62 22.3 mm to (335.0, 48.0)
- moved R63 22.3 mm to (335.0, 41.0)
- moved R83 22.2 mm to (335.0, 34.0)
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Connections:
- D1 pad 2: /DISCHARGE Top/CELL_18 -> Net-(D1-Pad2)
- D10 pad 2: /DISCHARGE Top/CELL_9 -> Net-(D10-Pad2)
- D11 pad 2: /DISCHARGE Top/CELL_8 -> Net-(D11-Pad2)
- D12 pad 2: /DISCHARGE Top/CELL_7 -> Net-(D12-Pad2)
- D13 pad 2: /DISCHARGE Top/CELL_6 -> Net-(D13-Pad2)
- D14 pad 2: /DISCHARGE Top/CELL_5 -> Net-(D14-Pad2)
- D15 pad 2: /DISCHARGE Top/CELL_4 -> Net-(D15-Pad2)
- D16 pad 2: /DISCHARGE Top/CELL_3 -> Net-(D16-Pad2)
- D17 pad 2: /DISCHARGE Top/CELL_2 -> Net-(D17-Pad2)
- D18 pad 2: /DISCHARGE Top/CELL_1 -> Net-(D18-Pad2)
- D2 pad 2: /DISCHARGE Top/CELL_16 -> Net-(D2-Pad2)
- D3 pad 2: /DISCHARGE Top/CELL_16 -> Net-(D3-Pad2)
- D4 pad 2: /DISCHARGE Top/CELL_15 -> Net-(D4-Pad2)
- D5 pad 2: /DISCHARGE Top/CELL_14 -> Net-(D5-Pad2)
- D6 pad 2: /DISCHARGE Top/CELL_13 -> Net-(D6-Pad2)
- D7 pad 2: /DISCHARGE Top/CELL_12 -> Net-(D7-Pad2)
- D8 pad 2: /DISCHARGE Top/CELL_11 -> Net-(D8-Pad2)
- D9 pad 2: /DISCHARGE Top/CELL_10 -> Net-(D9-Pad2)
- Q10 pad 3: Net-(Q10-Pad3) -> Net-(D9-Pad1)
- Q11 pad 3: Net-(Q11-Pad3) -> Net-(D10-Pad1)
- Q12 pad 3: Net-(Q12-Pad3) -> Net-(D11-Pad1)
- Q13 pad 3: Net-(Q13-Pad3) -> Net-(D12-Pad1)
- Q14 pad 3: Net-(Q14-Pad3) -> Net-(D13-Pad1)
- Q15 pad 3: Net-(Q15-Pad3) -> Net-(D14-Pad1)
- Q16 pad 3: Net-(Q16-Pad3) -> Net-(D15-Pad1)
- Q17 pad 3: Net-(Q17-Pad3) -> Net-(D16-Pad1)
- Q18 pad 3: Net-(Q18-Pad3) -> Net-(D17-Pad1)
- Q19 pad 3: Net-(Q19-Pad3) -> Net-(D18-Pad1)
- Q2 pad 3: Net-(Q2-Pad3) -> Net-(D1-Pad1)
- Q3 pad 3: Net-(Q3-Pad3) -> Net-(D2-Pad1)
- Q4 pad 3: Net-(Q4-Pad3) -> Net-(D3-Pad1)
- Q5 pad 3: Net-(Q5-Pad3) -> Net-(D4-Pad1)
- Q6 pad 3: Net-(Q6-Pad3) -> Net-(D5-Pad1)
- Q7 pad 3: Net-(Q7-Pad3) -> Net-(D6-Pad1)
- Q8 pad 3: Net-(Q8-Pad3) -> Net-(D7-Pad1)
- Q9 pad 3: Net-(Q9-Pad3) -> Net-(D8-Pad1)
- R33 pad 1: Net-(D1-Pad1) -> /DISCHARGE Top/CELL_18
- R33 pad 2: Net-(Q2-Pad3) -> Net-(D1-Pad2)
- R34 pad 1: Net-(D2-Pad1) -> /DISCHARGE Top/CELL_16
- R34 pad 2: Net-(Q3-Pad3) -> Net-(D2-Pad2)
- R35 pad 1: Net-(D3-Pad1) -> /DISCHARGE Top/CELL_16
- R35 pad 2: Net-(Q4-Pad3) -> Net-(D3-Pad2)
- R36 pad 1: Net-(D4-Pad1) -> /DISCHARGE Top/CELL_15
- R36 pad 2: Net-(Q5-Pad3) -> Net-(D4-Pad2)
- R37 pad 1: Net-(D5-Pad1) -> /DISCHARGE Top/CELL_14
- R37 pad 2: Net-(Q6-Pad3) -> Net-(D5-Pad2)
- R38 pad 1: Net-(D6-Pad1) -> /DISCHARGE Top/CELL_13
- R38 pad 2: Net-(Q7-Pad3) -> Net-(D6-Pad2)
- R39 pad 2: Net-(Q2-Pad3) -> Net-(D1-Pad1)
- R40 pad 2: Net-(Q3-Pad3) -> Net-(D2-Pad1)
- R41 pad 2: Net-(Q4-Pad3) -> Net-(D3-Pad1)
- R42 pad 2: Net-(Q5-Pad3) -> Net-(D4-Pad1)
- R43 pad 2: Net-(Q6-Pad3) -> Net-(D5-Pad1)
- R44 pad 2: Net-(Q7-Pad3) -> Net-(D6-Pad1)
- R58 pad 1: Net-(D7-Pad1) -> /DISCHARGE Top/CELL_12
- R58 pad 2: Net-(Q8-Pad3) -> Net-(D7-Pad2)
- R59 pad 1: Net-(D8-Pad1) -> /DISCHARGE Top/CELL_11
- R59 pad 2: Net-(Q9-Pad3) -> Net-(D8-Pad2)
- R60 pad 1: Net-(D9-Pad1) -> /DISCHARGE Top/CELL_10
- R60 pad 2: Net-(Q10-Pad3) -> Net-(D9-Pad2)
- R61 pad 1: Net-(D10-Pad1) -> /DISCHARGE Top/CELL_9
- R61 pad 2: Net-(Q11-Pad3) -> Net-(D10-Pad2)
- R62 pad 1: Net-(D11-Pad1) -> /DISCHARGE Top/CELL_8
- R62 pad 2: Net-(Q12-Pad3) -> Net-(D11-Pad2)
- R63 pad 1: Net-(D12-Pad1) -> /DISCHARGE Top/CELL_7
- R63 pad 2: Net-(Q13-Pad3) -> Net-(D12-Pad2)
- R64 pad 2: Net-(Q8-Pad3) -> Net-(D7-Pad1)
- R65 pad 2: Net-(Q9-Pad3) -> Net-(D8-Pad1)
- R66 pad 2: Net-(Q10-Pad3) -> Net-(D9-Pad1)
- R67 pad 2: Net-(Q11-Pad3) -> Net-(D10-Pad1)
- R68 pad 2: Net-(Q12-Pad3) -> Net-(D11-Pad1)
- R69 pad 2: Net-(Q13-Pad3) -> Net-(D12-Pad1)
- R83 pad 1: Net-(D13-Pad1) -> /DISCHARGE Top/CELL_6
- R83 pad 2: Net-(Q14-Pad3) -> Net-(D13-Pad2)
- R84 pad 1: Net-(D14-Pad1) -> /DISCHARGE Top/CELL_5
- R84 pad 2: Net-(Q15-Pad3) -> Net-(D14-Pad2)
- R85 pad 1: Net-(D15-Pad1) -> /DISCHARGE Top/CELL_4
- R85 pad 2: Net-(Q16-Pad3) -> Net-(D15-Pad2)
- R86 pad 1: Net-(D16-Pad1) -> /DISCHARGE Top/CELL_3
- R86 pad 2: Net-(Q17-Pad3) -> Net-(D16-Pad2)
- R87 pad 1: Net-(D17-Pad1) -> /DISCHARGE Top/CELL_2
- R87 pad 2: Net-(Q18-Pad3) -> Net-(D17-Pad2)
- R88 pad 1: Net-(D18-Pad1) -> /DISCHARGE Top/CELL_1
- R88 pad 2: Net-(Q19-Pad3) -> Net-(D18-Pad2)
- R89 pad 2: Net-(Q14-Pad3) -> Net-(D13-Pad1)
- R90 pad 2: Net-(Q15-Pad3) -> Net-(D14-Pad1)
- R91 pad 2: Net-(Q16-Pad3) -> Net-(D15-Pad1)
- R92 pad 2: Net-(Q17-Pad3) -> Net-(D16-Pad1)
- R93 pad 2: Net-(Q18-Pad3) -> Net-(D17-Pad1)
- R94 pad 2: Net-(Q19-Pad3) -> Net-(D18-Pad1)
Routing:
- net GND_1: track 0.00 -> 75.2 mm
- net /DISCHARGE Top/CELL_5: track 0.00 -> 54.0 mm
- net /DISCHARGE Top/CELL_1: track 0.00 -> 43.4 mm
- net /DISCHARGE Top/CELL_2: track 0.00 -> 41.7 mm
- net /DISCHARGE Top/CELL_3: track 0.00 -> 38.0 mm
- net /DISCHARGE Top/CELL_6: track 0.00 -> 31.5 mm
- net /DISCHARGE Top/CELL_4: track 0.00 -> 31.3 mm
- net /DISCHARGE Top/CELL_7: track 0.00 -> 26.2 mm
Other:
- board size 129.2 x 133.8 mm -> 69.8 x 133.3 mm
- net class Power added: clearance 0.2, trace_width 1.5, via_dia 2, via_drill 1.7

Commit message: more PCB layout work
Parts:
- added REF**: 3.5mm ISO, rLoop_Footprints:rLoop_mounting_hole_iso_3.5mm, F.Cu at (61.8, 171.0)
- added REF**: 3.5mm ISO, rLoop_Footprints:rLoop_mounting_hole_iso_3.5mm, F.Cu at (121.8, 171.0)
- added REF**: 3.5mm ISO, rLoop_Footprints:rLoop_mounting_hole_iso_3.5mm, F.Cu at (106.8, 171.0)
- added REF**: 3.5mm ISO, rLoop_Footprints:rLoop_mounting_hole_iso_3.5mm, F.Cu at (121.8, 121.0)
- added REF**: 3.5mm ISO, rLoop_Footprints:rLoop_mounting_hole_iso_3.5mm, F.Cu at (106.8, 121.0)
- added REF**: 3.5mm ISO, rLoop_Footprints:rLoop_mounting_hole_iso_3.5mm, F.Cu at (61.8, 121.0)
- added REF**: 3.5mm ISO, rLoop_Footprints:rLoop_mounting_hole_iso_3.5mm, F.Cu at (57.2, 51.5)
- added REF**: 3.5mm ISO, rLoop_Footprints:rLoop_mounting_hole_iso_3.5mm, F.Cu at (121.8, 80.5)
- J1: footprint Pin_Headers:Pin_Header_Straight_2x07_Pitch2.54mm_SMD -> rLoop_Footprints:Pin_Header_Straight_2x07_Pitch2.54mm_SMD_MIRROR; moved to B.Cu
- moved R16 250.9 mm to (66.0, 168.8), turned to 90 degrees
- moved R26 249.5 mm to (67.8, 168.8), turned to 90 degrees
- moved J2 248.2 mm to (115.5, 125.8)
- moved C29 245.4 mm to (56.2, 138.2), turned to 270 degrees
- moved R85 245.0 mm to (94.8, 65.2)
- moved R86 244.7 mm to (95.0, 58.2)
- moved R61 244.5 mm to (94.8, 100.2)
- moved R62 244.5 mm to (94.8, 93.2)
- moved R63 244.5 mm to (94.8, 86.2)
- moved R83 244.5 mm to (94.8, 79.2)
- moved R84 244.5 mm to (94.8, 72.2)
- moved R33 244.2 mm to (94.5, 163.8)
- moved R34 244.2 mm to (94.5, 156.8)
- moved R35 244.2 mm to (95.0, 149.8)
- moved R36 244.2 mm to (94.5, 142.8)
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Connections:
- J2 pad 3: /DISCHARGE Top/CELL_16 -> /DISCHARGE Top/CELL_17
- Q2 pad 2: /DISCHARGE Top/CELL_16 -> /DISCHARGE Top/CELL_17
- R27 pad 1: /DISCHARGE Top/CELL_16 -> /DISCHARGE Top/CELL_17
- R34 pad 1: /DISCHARGE Top/CELL_16 -> /DISCHARGE Top/CELL_17
- R40 pad 1: /DISCHARGE Top/CELL_16 -> /DISCHARGE Top/CELL_17
Routing:
- net /MCU Connector/MISO_TO_PWR_NODE: track 0.00 -> 130.3 mm, vias 0 -> 1
- net /MCU Connector/SCK_FROM_PWR_NODE: track 0.00 -> 127.9 mm, vias 0 -> 1
- net /MCU Connector/MOSI_FROM_PWR_NODE: track 0.00 -> 127.7 mm, vias 0 -> 1
- net /CONTROLLER 1/IRQ_OUT: track 0.00 -> 126.7 mm, vias 0 -> 1
- net /MCU Connector/NCS_FROM_PWR_NODE: track 0.00 -> 123.5 mm, vias 0 -> 1
- net /DISCHARGE Top/CELL_9: track 0.00 -> 63.7 mm, vias 0 -> 1
- net /DISCHARGE Top/CELL_8: track 0.00 -> 59.6 mm, vias 0 -> 1
- net /DISCHARGE Top/CELL_12: track 0.00 -> 59.0 mm, vias 0 -> 1
- net /DISCHARGE Top/CELL_10: track 0.00 -> 56.6 mm, vias 0 -> 1
- net /DISCHARGE Top/CELL_18: track 0.00 -> 54.8 mm
- net /DISCHARGE Top/CELL_11: track 0.00 -> 52.5 mm, vias 0 -> 1
- net /DISCHARGE Top/CELL_1: track 43.4 -> 92.6 mm, vias 0 -> 2
- net /DISCHARGE Top/CELL_6: track 31.5 -> 80.6 mm, vias 0 -> 1
- net /DISCHARGE Top/CELL_13: track 0.00 -> 47.5 mm, vias 0 -> 1
- net /DISCHARGE Top/CELL_14: track 0.00 -> 47.0 mm, vias 0 -> 1
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- added copper zone on B.Cu, net GND_1
- added copper zone on F.Cu, net GND_1
Other:
- board size 69.8 x 133.3 mm -> 77.5 x 133 mm
- board text added: "CHECK PN ON FLIP FLOP"
- board text added: "TODO: ADD JUMPER TO BYPASS OPTO ISOLATOR"
- board text added: "WRONG FOOTPRINT FOR OPTO"

Commit message: more PCB work on BMS v2
Parts:
- added R95: 10R / 0.125W / 1% / SMD 0603, Resistors_SMD:R_0603, F.Cu at (76.7, 45.6)
- U1: footprint Housings_DIP:DIP-4_W7.62mm -> rLoop_Footprints:VOS618A-2X001T
- moved C6 15.9 mm to (60.2, 89.1), turned to 0 degrees
- moved U1 14.4 mm to (54.6, 145.1)
- moved R7 13.9 mm to (58.2, 140.7), turned to 0 degrees
- moved R12 12.3 mm to (67.7, 82.0), turned to 90 degrees
- moved R88 9.36 mm to (85.9, 46.2)
- moved Q1 6.88 mm to (59.0, 144.1), turned to 180 degrees
- moved C5 4.35 mm to (58.0, 99.2)
- moved R6 4.22 mm to (57.6, 148.5), turned to 180 degrees
- moved C31 3.79 mm to (57.5, 135.8)
- moved R5 3.57 mm to (60.8, 147.1), turned to 0 degrees
- moved C33 3.36 mm to (64.0, 138.5), turned to 0 degrees
- moved C29 2.15 mm to (55.0, 136.5)
- moved R9 2.05 mm to (57.2, 96.0)
- moved C3 2.01 mm to (56.1, 100.0)
- moved R11 1.65 mm to (55.6, 91.4)
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Connections:
- J2 pad 20: GND_1 -> /DISCHARGE Top/CELL_0
- Q19 pad 2: GND_1 -> /DISCHARGE Top/CELL_0
- R82 pad 1: GND_1 -> /DISCHARGE Top/CELL_0
Routing:
- net /Clock Generator/VDD: track 0.00 -> 131.5 mm, vias 0 -> 1
- net /DISCHARGE Top/CELL_0: track 0.00 -> 79.4 mm
- net VDDHV_3: track 0.00 -> 59.8 mm
- net /CONTROLLER 3/VDDHVM: track 0.00 -> 50.3 mm
- net /CONTROLLER 2/~PD_IN: track 0.00 -> 49.5 mm
- net /CONTROLLER 2/VDDHVM: track 0.00 -> 45.5 mm
- net /CONTROLLER 1/~PD_IN: track 0.00 -> 43.6 mm
- net GND_2: track 2.50 -> 35.9 mm, vias 2 -> 11
- net GND_1: track 96.3 -> 129.3 mm, vias 4 -> 15
- net GND_3: track 9.50 -> 42.4 mm, vias 0 -> 10
- net MCU_3V3: track 35.6 -> 3.95 mm
- net Net-(C19-Pad2): track 0.00 -> 24.9 mm, vias 0 -> 2
- net /MCU Connector/POWER_DN_DISABLE_FROM_PWR_NODE: track 0.00 -> 19.7 mm, vias 0 -> 1
- net MCU_GND: track 0.00 -> 16.8 mm, vias 0 -> 1
- net Net-(C6-Pad2): track 0.00 -> 14.9 mm, vias 0 -> 2
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- added copper zone on B.Cu, net GND_2
- added copper zone on F.Cu, net GND_2
- added copper zone on B.Cu, net GND_3
- added copper zone on F.Cu, net GND_3
Other:
- net class Default: clearance 0.2 -> 0.1524; via_dia 0.6 -> 0.6858; via_drill 0.4 -> 0.3302
- net class Power: trace_width 1.5 -> 1.2
- rule trace_clearance: 0.2 -> 0.1524
- rule trace_min: 0.2 -> 0.1524
- rule via_min_drill: 0.3 -> 0.3302
- rule via_min_size: 0.4 -> 0.6858
- board text removed: "CHECK PN ON FLIP FLOP"
- board text removed: "WRONG FOOTPRINT FOR OPTO"
