File: RLOOP_BMS_V2/DISCHARGE Top.sch (KiCad schematic (older format))
At the start: 111 parts, among them Q10 PMV20ENR, Q11 PMV20ENR, Q12 PMV20ENR, Q13 PMV20ENR, Q14 PMV20ENR, Q15 PMV20ENR, Q16 PMV20ENR, Q17 PMV20ENR, Q18 PMV20ENR, Q19 PMV20ENR, Q2 PMV20ENR, Q3 PMV20ENR, Q4 PMV20ENR, Q5 PMV20ENR, Q6 PMV20ENR, Q7 PMV20ENR, Q8 PMV20ENR, Q9 PMV20ENR

Commit message: Footprint work
starting to assign footprints to parts
Parts:
- D1, D10, D11, D12, D13, D14, D15, D16, D17, D18, D2, D3, D4, D5, D6, D7, D8, D9: footprint (none) -> LEDs:LED_0805
- R20, R21, R22, R23, R24, R25, R26, R27, R28, R29, R30, R31, R32, R33, R34, R35, R36, R37, R38, R45, R46, R47, R48, R49, R50, R51, R52, R53, R54, R55, R56, R57, R58, R59, R60, R61, R62, R63, R70, R71, R72, R73, R74, R75, R76, R77, R78, R79, R80, R81, R82, R83, R84, R85, R86, R87, R88: footprint (none) -> Resistors_SMD:R_0603

Commit message: footprint and layout work WIP
Parts:
- Q10, Q11, Q12, Q13, Q14, Q15, Q16, Q17, Q18, Q19, Q2, Q3, Q4, Q5, Q6, Q7, Q8, Q9: footprint (none) -> rLoop_Footprints:PMV20ENR-TO_236AB
- R39, R40, R41, R42, R43, R44, R64, R65, R66, R67, R68, R69, R89, R90, R91, R92, R93, R94: footprint (none) -> TO_SOT_Packages_THT:TO-220-2_Vertical
Changed lines of the file:
@@
 F 0 "R39" V 3130 1800 50  0000 C CNN
 F 1 "MP930-2.00-1%" V 3200 1800 50  0000 C CNN
-F 2 "" V 2980 1800 50  0001 C CNN
+F 2 "TO_SOT_Packages_THT:TO-220-2_Vertical" V 2980 1800 50  0001 C CNN
 F 3 "" H 3050 1800 50  0001 C CNN
 	1    3050 1800
@@
 F 0 "R40" V 3130 2600 50  0000 C CNN
 F 1 "MP930-2.00-1%" V 3200 2600 50  0000 C CNN
-F 2 "" V 2980 2600 50  0001 C CNN
+F 2 "TO_SOT_Packages_THT:TO-220-2_Vertical" V 2980 2600 50  0001 C CNN
 F 3 "" H 3050 2600 50  0001 C CNN
 	1    3050 2600
@@
 F 0 "R41" V 3130 3400 50  0000 C CNN
 F 1 "MP930-2.00-1%" V 3200 3400 50  0000 C CNN
-F 2 "" V 2980 3400 50  0001 C CNN
+F 2 "TO_SOT_Packages_THT:TO-220-2_Vertical" V 2980 3400 50  0001 C CNN
 F 3 "" H 3050 3400 50  0001 C CNN
 	1    3050 3400
@@
 F 0 "R42" V 3130 4200 50  0000 C CNN
 F 1 "MP930-2.00-1%" V 3200 4200 50  0000 C CNN
-F 2 "" V 2980 4200 50  0001 C CNN
+F 2 "TO_SOT_Packages_THT:TO-220-2_Vertical" V 2980 4200 50  0001 C CNN
 F 3 "" H 3050 4200 50  0001 C CNN
 	1    3050 4200
@@
 F 0 "R43" V 3130 5000 50  0000 C CNN
 F 1 "MP930-2.00-1%" V 3200 5000 50  0000 C CNN
-F 2 "" V 2980 5000 50  0001 C CNN
+F 2 "TO_SOT_Packages_THT:TO-220-2_Vertical" V 2980 5000 50  0001 C CNN
 F 3 "" H 3050 5000 50  0001 C CNN
 	1    3050 5000
@@
 F 0 "R44" V 3130 5800 50  0000 C CNN
 F 1 "MP930-2.00-1%" V 3200 5800 50  0000 C CNN
-F 2 "" V 2980 5800 50  0001 C CNN
+F 2 "TO_SOT_Packages_THT:TO-220-2_Vertical" V 2980 5800 50  0001 C CNN
 F 3 "" H 3050 5800 50  0001 C CNN
 	1    3050 5800
@@
 F 0 "R64" V 6530 1800 50  0000 C CNN
 F 1 "MP930-2.00-1%" V 6600 1800 50  0000 C CNN
-F 2 "" V 6380 1800 50  0001 C CNN
+F 2 "TO_SOT_Packages_THT:TO-220-2_Vertical" V 6380 1800 50  0001 C CNN
 F 3 "" H 6450 1800 50  0001 C CNN
 	1    6450 1800
@@
 F 0 "R65" V 6530 2600 50  0000 C CNN
 F 1 "MP930-2.00-1%" V 6600 2600 50  0000 C CNN
-F 2 "" V 6380 2600 50  0001 C CNN
+F 2 "TO_SOT_Packages_THT:TO-220-2_Vertical" V 6380 2600 50  0001 C CNN
 F 3 "" H 6450 2600 50  0001 C CNN
 	1    6450 2600
@@
 F 0 "R66" V 6530 3400 50  0000 C CNN
 F 1 "MP930-2.00-1%" V 6600 3400 50  0000 C CNN
-F 2 "" V 6380 3400 50  0001 C CNN
+F 2 "TO_SOT_Packages_THT:TO-220-2_Vertical" V 6380 3400 50  0001 C CNN
 F 3 "" H 6450 3400 50  0001 C CNN
 	1    6450 3400
@@
 F 0 "R67" V 6530 4200 50  0000 C CNN
 F 1 "MP930-2.00-1%" V 6600 4200 50  0000 C CNN
-F 2 "" V 6380 4200 50  0001 C CNN
+F 2 "TO_SOT_Packages_THT:TO-220-2_Vertical" V 6380 4200 50  0001 C CNN
 F 3 "" H 6450 4200 50  0001 C CNN
 	1    6450 4200
@@
 F 0 "R68" V 6530 5000 50  0000 C CNN
 F 1 "MP930-2.00-1%" V 6600 5000 50  0000 C CNN
-F 2 "" V 6380 5000 50  0001 C CNN
+F 2 "TO_SOT_Packages_THT:TO-220-2_Vertical" V 6380 5000 50  0001 C CNN
 F 3 "" H 6450 5000 50  0001 C CNN
 	1    6450 5000
@@
 F 0 "R69" V 6530 5800 50  0000 C CNN
 F 1 "MP930-2.00-1%" V 6600 5800 50  0000 C CNN
-F 2 "" V 6380 5800 50  0001 C CNN
+F 2 "TO_SOT_Packages_THT:TO-220-2_Vertical" V 6380 5800 50  0001 C CNN
 F 3 "" H 6450 5800 50  0001 C CNN
 	1    6450 5800
@@
 F 0 "R89" V 9880 1800 50  0000 C CNN
 F 1 "MP930-2.00-1%" V 9950 1800 50  0000 C CNN
-F 2 "" V 9730 1800 50  0001 C CNN
+F 2 "TO_SOT_Packages_THT:TO-220-2_Vertical" V 9730 1800 50  0001 C CNN
 F 3 "" H 9800 1800 50  0001 C CNN
 	1    9800 1800
@@
 F 0 "R90" V 9880 2600 50  0000 C CNN
 F 1 "MP930-2.00-1%" V 9950 2600 50  0000 C CNN
-F 2 "" V 9730 2600 50  0001 C CNN
+F 2 "TO_SOT_Packages_THT:TO-220-2_Vertical" V 9730 2600 50  0001 C CNN
 F 3 "" H 9800 2600 50  0001 C CNN
 	1    9800 2600
@@
 F 0 "R91" V 9880 3400 50  0000 C CNN
 F 1 "MP930-2.00-1%" V 9950 3400 50  0000 C CNN
-F 2 "" V 9730 3400 50  0001 C CNN
+F 2 "TO_SOT_Packages_THT:TO-220-2_Vertical" V 9730 3400 50  0001 C CNN
 F 3 "" H 9800 3400 50  0001 C CNN
 	1    9800 3400
@@
 F 0 "R92" V 9880 4200 50  0000 C CNN
 F 1 "MP930-2.00-1%" V 9950 4200 50  0000 C CNN
-F 2 "" V 9730 4200 50  0001 C CNN
+F 2 "TO_SOT_Packages_THT:TO-220-2_Vertical" V 9730 4200 50  0001 C CNN
 F 3 "" H 9800 4200 50  0001 C CNN
 	1    9800 4200
@@
 F 0 "R93" V 9880 5000 50  0000 C CNN
 F 1 "MP930-2.00-1%" V 9950 5000 50  0000 C CNN
-F 2 "" V 9730 5000 50  0001 C CNN
+F 2 "TO_SOT_Packages_THT:TO-220-2_Vertical" V 9730 5000 50  0001 C CNN
 F 3 "" H 9800 5000 50  0001 C CNN
 	1    9800 5000
@@
 F 0 "R94" V 9880 5800 50  0000 C CNN
 F 1 "MP930-2.00-1%" V 9950 5800 50  0000 C CNN
-F 2 "" V 9730 5800 50  0001 C CNN
+F 2 "TO_SOT_Packages_THT:TO-220-2_Vertical" V 9730 5800 50  0001 C CNN
 F 3 "" H 9800 5800 50  0001 C CNN
 	1    9800 5800
@@
 F 0 "Q2" H 2200 1750 50  0000 L CNN
 F 1 "PMV20ENR" H 2200 1650 50  0000 L CNN
-F 2 "" H 2200 1900 50  0001 C CNN
+F 2 "rLoop_Footprints:PMV20ENR-TO_236AB" H 2200 1900 50  0001 C CNN
 F 3 "" H 2000 1800 50  0001 C CNN
 	1    2000 1800
@@
 F 0 "Q3" H 2200 2550 50  0000 L CNN
 F 1 "PMV20ENR" H 2200 2450 50  0000 L CNN
-F 2 "" H 2200 2700 50  0001 C CNN
+F 2 "rLoop_Footprints:PMV20ENR-TO_236AB" H 2200 2700 50  0001 C CNN
 F 3 "" H 2000 2600 50  0001 C CNN
 	1    2000 2600
@@
 F 0 "Q4" H 2200 3350 50  0000 L CNN
 F 1 "PMV20ENR" H 2200 3250 50  0000 L CNN
-F 2 "" H 2200 3500 50  0001 C CNN
+F 2 "rLoop_Footprints:PMV20ENR-TO_236AB" H 2200 3500 50  0001 C CNN
 F 3 "" H 2000 3400 50  0001 C CNN
 	1    2000 3400
@@
 F 0 "Q5" H 2200 4150 50  0000 L CNN
 F 1 "PMV20ENR" H 2200 4050 50  0000 L CNN
-F 2 "" H 2200 4300 50  0001 C CNN
+F 2 "rLoop_Footprints:PMV20ENR-TO_236AB" H 2200 4300 50  0001 C CNN
 F 3 "" H 2000 4200 50  0001 C CNN
 	1    2000 4200
@@
 F 0 "Q6" H 2200 4950 50  0000 L CNN
 F 1 "PMV20ENR" H 2200 4850 50  0000 L CNN
-F 2 "" H 2200 5100 50  0001 C CNN
+F 2 "rLoop_Footprints:PMV20ENR-TO_236AB" H 2200 5100 50  0001 C CNN
 F 3 "" H 2000 5000 50  0001 C CNN
 	1    2000 5000
@@
 F 0 "Q7" H 2200 5750 50  0000 L CNN
 F 1 "PMV20ENR" H 2200 5650 50  0000 L CNN
-F 2 "" H 2200 5900 50  0001 C CNN
+F 2 "rLoop_Footprints:PMV20ENR-TO_236AB" H 2200 5900 50  0001 C CNN
 F 3 "" H 2000 5800 50  0001 C CNN
 	1    2000 5800
@@
 F 0 "Q13" H 5600 5750 50  0000 L CNN
 F 1 "PMV20ENR" H 5600 5650 50  0000 L CNN
-F 2 "" H 5600 5900 50  0001 C CNN
+F 2 "rLoop_Footprints:PMV20ENR-TO_236AB" H 5600 5900 50  0001 C CNN
 F 3 "" H 5400 5800 50  0001 C CNN
 	1    5400 5800
@@
 F 0 "Q12" H 5600 4950 50  0000 L CNN
 F 1 "PMV20ENR" H 5600 4850 50  0000 L CNN
-F 2 "" H 5600 5100 50  0001 C CNN
+F 2 "rLoop_Footprints:PMV20ENR-TO_236AB" H 5600 5100 50  0001 C CNN
 F 3 "" H 5400 5000 50  0001 C CNN
 	1    5400 5000
@@
 F 0 "Q11" H 5600 4150 50  0000 L CNN
 F 1 "PMV20ENR" H 5600 4050 50  0000 L CNN
-F 2 "" H 5600 4300 50  0001 C CNN
+F 2 "rLoop_Footprints:PMV20ENR-TO_236AB" H 5600 4300 50  0001 C CNN
 F 3 "" H 5400 4200 50  0001 C CNN
 	1    5400 4200
@@
 F 0 "Q10" H 5600 3350 50  0000 L CNN
 F 1 "PMV20ENR" H 5600 3250 50  0000 L CNN
-F 2 "" H 5600 3500 50  0001 C CNN
+F 2 "rLoop_Footprints:PMV20ENR-TO_236AB" H 5600 3500 50  0001 C CNN
 F 3 "" H 5400 3400 50  0001 C CNN
 	1    5400 3400
@@
 F 0 "Q9" H 5600 2550 50  0000 L CNN
 F 1 "PMV20ENR" H 5600 2450 50  0000 L CNN
-F 2 "" H 5600 2700 50  0001 C CNN
+F 2 "rLoop_Footprints:PMV20ENR-TO_236AB" H 5600 2700 50  0001 C CNN
 F 3 "" H 5400 2600 50  0001 C CNN
 	1    5400 2600
@@
 F 0 "Q8" H 5600 1750 50  0000 L CNN
 F 1 "PMV20ENR" H 5600 1650 50  0000 L CNN
-F 2 "" H 5600 1900 50  0001 C CNN
+F 2 "rLoop_Footprints:PMV20ENR-TO_236AB" H 5600 1900 50  0001 C CNN
 F 3 "" H 5400 1800 50  0001 C CNN
 	1    5400 1800
@@
 F 0 "Q14" H 8950 1750 50  0000 L CNN
 F 1 "PMV20ENR" H 8950 1650 50  0000 L CNN
-F 2 "" H 8950 1900 50  0001 C CNN
+F 2 "rLoop_Footprints:PMV20ENR-TO_236AB" H 8950 1900 50  0001 C CNN
 F 3 "" H 8750 1800 50  0001 C CNN
 	1    8750 1800
@@
 F 0 "Q15" H 8950 2550 50  0000 L CNN
 F 1 "PMV20ENR" H 8950 2450 50  0000 L CNN
-F 2 "" H 8950 2700 50  0001 C CNN
+F 2 "rLoop_Footprints:PMV20ENR-TO_236AB" H 8950 2700 50  0001 C CNN
 F 3 "" H 8750 2600 50  0001 C CNN
 	1    8750 2600
@@
 F 0 "Q16" H 8950 3350 50  0000 L CNN
 F 1 "PMV20ENR" H 8950 3250 50  0000 L CNN
-F 2 "" H 8950 3500 50  0001 C CNN
+F 2 "rLoop_Footprints:PMV20ENR-TO_236AB" H 8950 3500 50  0001 C CNN
 F 3 "" H 8750 3400 50  0001 C CNN
 	1    8750 3400
@@
 F 0 "Q17" H 8950 4150 50  0000 L CNN
 F 1 "PMV20ENR" H 8950 4050 50  0000 L CNN
-F 2 "" H 8950 4300 50  0001 C CNN
+F 2 "rLoop_Footprints:PMV20ENR-TO_236AB" H 8950 4300 50  0001 C CNN
 F 3 "" H 8750 4200 50  0001 C CNN
 	1    8750 4200
@@
 F 0 "Q18" H 8950 4950 50  0000 L CNN
 F 1 "PMV20ENR" H 8950 4850 50  0000 L CNN
-F 2 "" H 8950 5100 50  0001 C CNN
+F 2 "rLoop_Footprints:PMV20ENR-TO_236AB" H 8950 5100 50  0001 C CNN
 F 3 "" H 8750 5000 50  0001 C CNN
 	1    8750 5000
@@
 F 0 "Q19" H 8950 5750 50  0000 L CNN
 F 1 "PMV20ENR" H 8950 5650 50  0000 L CNN
-F 2 "" H 8950 5900 50  0001 C CNN
+F 2 "rLoop_Footprints:PMV20ENR-TO_236AB" H 8950 5900 50  0001 C CNN
 F 3 "" H 8750 5800 50  0001 C CNN
 	1    8750 5800

Commit message: PCB Layout WIP
Parts:
- R39, R40, R41, R42, R43, R44, R64, R65, R66, R67, R68, R69, R89, R90, R91, R92, R93, R94: footprint TO_SOT_Packages_THT:TO-220-2_Vertical -> rLoop_Footprints:Res_MP930
Connections:
- net CELL_1: now also R88.1; no longer D18.2 (A)
- net CELL_10: now also R60.1; no longer D9.2 (A)
- net CELL_11: now also R59.1; no longer D8.2 (A)
- net CELL_12: now also R58.1; no longer D7.2 (A)
- net CELL_13: now also R38.1; no longer D6.2 (A)
- net CELL_14: now also R37.1; no longer D5.2 (A)
- net CELL_15: now also R36.1; no longer D4.2 (A)
- net CELL_16: now also R35.1; no longer D3.2 (A)
- net CELL_17: now also R34.1; no longer D2.2 (A)
- net CELL_18: now also R33.1; no longer D1.2 (A)
- net CELL_2: now also R87.1; no longer D17.2 (A)
- net CELL_3: now also R86.1; no longer D16.2 (A)
- net CELL_4: now also R85.1; no longer D15.2 (A)
- net CELL_5: now also R84.1; no longer D14.2 (A)
- net CELL_6: now also R83.1; no longer D13.2 (A)
- net CELL_7: now also R63.1; no longer D12.2 (A)
- net CELL_8: now also R62.1; no longer D11.2 (A)
- net CELL_9: now also R61.1; no longer D10.2 (A)
- net at D2.1 (K): now also Q3.3 (D), R40.2; no longer R34.1
- net at D3.1 (K): now also Q4.3 (D), R41.2; no longer R35.1
- net at D4.1 (K): now also Q5.3 (D), R42.2; no longer R36.1
- net at D5.1 (K): now also Q6.3 (D), R43.2; no longer R37.1
- net at D6.1 (K): now also Q7.3 (D), R44.2; no longer R38.1
- net at D7.1 (K): now also Q8.3 (D), R64.2; no longer R58.1
- net at D8.1 (K): now also Q9.3 (D), R65.2; no longer R59.1
- net at D9.1 (K): now also Q10.3 (D), R66.2; no longer R60.1
- net at D10.1 (K): now also Q11.3 (D), R67.2; no longer R61.1
- net at D11.1 (K): now also Q12.3 (D), R68.2; no longer R62.1
- net at D12.1 (K): now also Q13.3 (D), R69.2; no longer R63.1
- net at D13.1 (K): now also Q14.3 (D), R89.2; no longer R83.1
- net at D14.1 (K): now also Q15.3 (D), R90.2; no longer R84.1
- net at D15.1 (K): now also Q16.3 (D), R91.2; no longer R85.1
- net at D16.1 (K): now also Q17.3 (D), R92.2; no longer R86.1
- net at D17.1 (K): now also Q18.3 (D), R93.2; no longer R87.1
- net at D18.1 (K): now also Q19.3 (D), R94.2; no longer R88.1
- net at Q2.3 (D), R39.2: now also D1.1 (K); no longer R33.2
- new net: D2.2 (A), R34.2
- new net: D3.2 (A), R35.2
- new net: D4.2 (A), R36.2
- new net: D5.2 (A), R37.2
- new net: D6.2 (A), R38.2
- new net: D7.2 (A), R58.2
- new net: D8.2 (A), R59.2
- new net: D9.2 (A), R60.2
- new net: D10.2 (A), R61.2
- new net: D11.2 (A), R62.2
- new net: D12.2 (A), R63.2
- new net: D13.2 (A), R83.2
- new net: D14.2 (A), R84.2
- new net: D15.2 (A), R85.2
- new net: D16.2 (A), R86.2
- new net: D17.2 (A), R87.2
- new net: D18.2 (A), R88.2
- new net: D1.2 (A), R33.2
Other:
- moved on the sheet: D1, D10, D11, D12, D13, D14, D15, D16, D17, D18, D2, D3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
