File: RLOOP_BMS_V2/CONTROLLER_1.sch (KiCad schematic (older format))
At the start: 27 parts, among them U3 bq76PL536A_HTQFP

Commit message: More BMS v2.5 WIP
Parts:
- R120, R121, R122, R123: renamed from R?; footprint (none) -> Resistors_SMD:R_0603
- TH5, TH6: renamed from TH?; footprint (none) -> Resistors_SMD:R_0603
- gave numbers to parts that had none: 2
Changed lines of the file:
@@
 $Descr A4 11693 8268
 encoding utf-8
-Sheet 6 9
+Sheet 6 10
 Title ""
 Date ""
@@
 Connection ~ 2700 3350
 $Comp
-L C C?
+L C C63
 U 1 1 592E9B54
 P 3750 1650
-F 0 "C?" H 3775 1750 50  0000 L CNN
+F 0 "C63" H 3775 1750 50  0000 L CNN
 F 1 ".047 uF / 50V/ 10% / SMD 0603" H 3800 1850 50  0000 L CNN
 F 2 "Capacitors_SMD:C_0603" H 3788 1500 50  0001 C CNN
@@
 $EndComp
 $Comp
-L R R?
+L R R123
 U 1 1 592E9D33
 P 4000 2250
-F 0 "R?" V 3900 2250 50  0000 C CNN
+F 0 "R123" V 3900 2250 50  0000 C CNN
 F 1 "1.82k / 0.063W / 1% / SMD0603" V 3750 2750 50  0000 C CNN
-F 2 "" V 3930 2250 50  0001 C CNN
+F 2 "Resistors_SMD:R_0603" V 3930 2250 50  0001 C CNN
 F 3 "" H 4000 2250 50  0001 C CNN
 	1    4000 2250
@@
 $EndComp
 $Comp
-L R R?
+L R R122
 U 1 1 592E9EB3
 P 3500 2250
-F 0 "R?" V 3580 2250 50  0000 C CNN
+F 0 "R122" V 3580 2250 50  0000 C CNN
 F 1 "1.47k / 0.063W / 1% / SMD0603" V 3650 2250 50  0000 C CNN
-F 2 "" V 3430 2250 50  0001 C CNN
+F 2 "Resistors_SMD:R_0603" V 3430 2250 50  0001 C CNN
 F 3 "" H 3500 2250 50  0001 C CNN
 	1    3500 2250
@@
 $EndComp
 $Comp
-L Thermistor_NTC TH?
+L Thermistor_NTC TH6
 U 1 1 592E9FE1
 P 3250 1650
-F 0 "TH?" H 3000 1700 50  0000 C CNN
+F 0 "TH6" H 3000 1700 50  0000 C CNN
 F 1 "10k / 1% / 3454K / SMD0603" H 2450 1600 50  0000 C CNN
-F 2 "" H 3250 1700 50  0001 C CNN
+F 2 "Resistors_SMD:R_0603" H 3250 1700 50  0001 C CNN
 F 3 "" H 3250 1700 50  0001 C CNN
 	1    3250 1650
@@
 Connection ~ 3250 1350
 $Comp
-L C C?
+L C C62
 U 1 1 592EAB7E
 P 2650 4750
-F 0 "C?" H 2675 4850 50  0000 L CNN
+F 0 "C62" H 2675 4850 50  0000 L CNN
 F 1 ".047 uF / 50V/ 10% / SMD 0603" H 2850 4750 50  0000 L CNN
 F 2 "Capacitors_SMD:C_0603" H 2688 4600 50  0001 C CNN
@@
 $EndComp
 $Comp
-L R R?
+L R R120
 U 1 1 592EABDC
 P 2300 4450
-F 0 "R?" V 2200 4450 50  0000 C CNN
+F 0 "R120" V 2200 4450 50  0000 C CNN
 F 1 "1.47k / 0.063W / 1% / SMD0603" V 2100 4150 50  0000 C CNN
-F 2 "" V 2230 4450 50  0001 C CNN
+F 2 "Resistors_SMD:R_0603" V 2230 4450 50  0001 C CNN
 F 3 "" H 2300 4450 50  0001 C CNN
 	1    2300 4450
@@
 $EndComp
 $Comp
-L R R?
+L R R121
 U 1 1 592EAC3F
 P 3000 4450
-F 0 "R?" V 3050 4650 50  0000 C CNN
+F 0 "R121" V 3050 4650 50  0000 C CNN
 F 1 "1.82k / 0.063W / 1% / SMD0603" V 3150 5050 50  0000 C CNN
-F 2 "" V 2930 4450 50  0001 C CNN
+F 2 "Resistors_SMD:R_0603" V 2930 4450 50  0001 C CNN
 F 3 "" H 3000 4450 50  0001 C CNN
 	1    3000 4450
@@
 $EndComp
 $Comp
-L Thermistor_NTC TH?
+L Thermistor_NTC TH5
 U 1 1 592EACA5
 P 1950 4800
-F 0 "TH?" H 1700 4850 50  0000 C CNN
+F 0 "TH5" H 1700 4850 50  0000 C CNN
 F 1 "10k / 1% / 3454K / SMD0603" H 1150 4750 50  0000 C CNN
-F 2 "" H 1950 4850 50  0001 C CNN
+F 2 "Resistors_SMD:R_0603" H 1950 4850 50  0001 C CNN
 F 3 "" H 1950 4850 50  0001 C CNN
 	1    1950 4800

Commit message: more WIP
TODO:
Fix pin 50
ground planes
figure out GND_2 weirdness
fix optoisolator 3d model
bq IC 3d model
triple check everything
BOM
Parts:
- added C76, C77: 33 pF / 50V/ 10% / SMD 0603, Capacitors_SMD:C_0603, symbol C
Connections:
- net DRDY_N: now also C77.1
- net SDO_N: now also C76.1
- net VDDHV_1: now also C76.2, C77.2
