File: RLOOP_BMS_V2/CONTROLLER_3.sch (KiCad schematic (older format))
At the start: 28 parts, among them U1 bq76PL536A_HTQFP

Commit message: More BMS v2.5 WIP
Parts:
- R112, R113, R114, R115: renamed from R?; footprint (none) -> Resistors_SMD:R_0603
- TH1, TH2: renamed from TH?; footprint (none) -> Resistors_SMD:R_0603
- gave numbers to parts that had none: 2
Changed lines of the file:
@@
 $Descr A4 11693 8268
 encoding utf-8
-Sheet 4 9
+Sheet 4 10
 Title ""
 Date ""
@@
 	9550 3700 9550 3900
 Wire Wire Line
-	6550 2050 9550 2050
-Wire Wire Line
-	9550 2050 9800 2050
+	6550 2050 9800 2050
 Wire Wire Line
 	9800 2150 6550 2150
 Wire Wire Line
-	6550 2250 9050 2250
-Wire Wire Line
-	9050 2250 9800 2250
+	6550 2250 9800 2250
 Wire Wire Line
 	9800 2350 6550 2350
 Wire Wire Line
-	6550 2450 8600 2450
-Wire Wire Line
-	8600 2450 9800 2450
+	6550 2450 9800 2450
 Wire Wire Line
 	6550 2550 9800 2550
 Wire Wire Line
-	6550 2650 8150 2650
-Wire Wire Line
-	8150 2650 9800 2650
+	6550 2650 9800 2650
 Wire Wire Line
 	6550 2750 9800 2750
 Wire Wire Line
-	6550 2850 7700 2850
-Wire Wire Line
-	7700 2850 9800 2850
+	6550 2850 9800 2850
 Wire Wire Line
 	6550 2950 9800 2950
 Wire Wire Line
-	6550 3050 7250 3050
-Wire Wire Line
-	7250 3050 9800 3050
+	6550 3050 9800 3050
 Wire Wire Line
 	6550 3150 9800 3150
@@
 Connection ~ 7250 3050
 Wire Wire Line
-	6550 1850 6650 1850
-Wire Wire Line
-	6650 1850 7350 1850
-Wire Wire Line
-	7350 1850 7600 1850
+	6550 1850 7600 1850
 Wire Wire Line
 	6550 1950 6650 1950
@@
 NoConn ~ 5400 4350
 Wire Wire Line
-	3950 2250 4150 2250
-Wire Wire Line
-	4150 2250 4300 2250
+	3950 2250 4300 2250
 Wire Wire Line
 	4150 2350 4300 2350
@@
 	6550 3500 6850 3500
 Wire Wire Line
-	6850 3500 6850 3600
-Wire Wire Line
-	6850 3600 6850 4000
-Wire Wire Line
-	6850 4000 6850 4150
+	6850 3500 6850 4150
 Wire Wire Line
 	6550 3600 6850 3600
@@
 GND_3
 Wire Wire Line
-	3950 2800 4200 2800
-Wire Wire Line
-	4200 2800 4300 2800
+	3950 2800 4300 2800
 Wire Wire Line
 	4300 2900 4200 2900
 Wire Wire Line
-	4200 2800 4200 2900
-Wire Wire Line
-	4200 2900 4200 3000
+	4200 2800 4200 3000
 Connection ~ 4200 2800
 Wire Wire Line
@@
 VDDHV_3
 Wire Wire Line
-	5100 1050 5200 1050
-Wire Wire Line
-	5200 1050 5300 1050
-Wire Wire Line
-	5300 1050 5400 1050
-Wire Wire Line
-	5400 1050 5500 1050
-Wire Wire Line
-	5500 1050 5600 1050
-Wire Wire Line
-	5600 1050 5700 1050
-Wire Wire Line
-	5700 1050 5800 1050
-Wire Wire Line
-	5800 1050 6000 1050
+	5100 1050 6000 1050
 Wire Wire Line
 	5100 1050 5100 1250
@@
 5V_3
 Wire Wire Line
-	3100 2600 3400 2600
-Wire Wire Line
-	3400 2600 4300 2600
+	3100 2600 4300 2600
 Text GLabel 4250 3450 0    60   Input ~ 0
 GND_3
@@
 	6550 1600 6750 1600
 Wire Wire Line
-	6750 1350 6750 1600
-Wire Wire Line
-	6750 1600 6750 1700
+	6750 1350 6750 1700
 Wire Wire Line
 	6750 1700 6550 1700
@@
 	2500 2500 2500 2600
 Wire Wire Line
-	2350 2600 2500 2600
-Wire Wire Line
-	2500 2600 2750 2600
+	2350 2600 2750 2600
 Wire Wire Line
 	2750 2600 2750 2500
@@
 	2750 2150 2750 2200
 Wire Wire Line
-	2300 2150 2500 2150
-Wire Wire Line
-	2500 2150 2750 2150
-Wire Wire Line
-	2750 2150 4300 2150
+	2300 2150 4300 2150
 Wire Wire Line
 	2500 2200 2500 2150
@@
 	4150 1950 4150 1850
 Wire Wire Line
-	2200 1850 2550 1850
-Wire Wire Line
-	2550 1850 4150 1850
-Wire Wire Line
-	4150 1850 4300 1850
+	2200 1850 4300 1850
 Wire Wire Line
 	2200 1850 2200 1600
@@
 	2550 1150 2550 1450
 Wire Wire Line
-	2100 1150 2200 1150
-Wire Wire Line
-	2200 1150 2550 1150
+	2100 1150 2550 1150
 Wire Wire Line
 	2200 1300 2200 1150
@@
 	4600 5200 4600 5500
 $Comp
-L C C?
+L C C59
 U 1 1 592E347D
 P 3800 950
-F 0 "C?" H 3825 1050 50  0000 L CNN
+F 0 "C59" H 3825 1050 50  0000 L CNN
 F 1 ".047 uF / 50V/ 10% / SMD 0603" H 3950 950 50  0000 L CNN
 F 2 "Capacitors_SMD:C_0603" H 3838 800 50  0001 C CNN
@@
 $EndComp
 $Comp
-L R R?
+L R R115
 U 1 1 592E3631
 P 4000 1500
-F 0 "R?" V 3900 1500 50  0000 C CNN
+F 0 "R115" V 3900 1500 50  0000 C CNN
 F 1 "1.82k / 0.063W / 1% / SMD 0603" V 3800 1850 50  0000 C CNN
-F 2 "" V 3930 1500 50  0001 C CNN
+F 2 "Resistors_SMD:R_0603" V 3930 1500 50  0001 C CNN
 F 3 "" H 4000 1500 50  0001 C CNN
 	1    4000 1500
@@
 $EndComp
 $Comp
-L R R?
+L R R114
 U 1 1 592E39D7
 P 3550 1500
-F 0 "R?" V 3650 1500 50  0000 C CNN
+F 0 "R114" V 3650 1500 50  0000 C CNN
 F 1 "1.47k / 0.063W / 1% / SMD 0603" V 3750 1600 50  0000 C CNN
-F 2 "" V 3480 1500 50  0001 C CNN
+F 2 "Resistors_SMD:R_0603" V 3480 1500 50  0001 C CNN
 F 3 "" H 3550 1500 50  0001 C CNN
 	1    3550 1500
@@
 $EndComp
 $Comp
-L Thermistor_NTC TH?
+L Thermistor_NTC TH2
 U 1 1 592E3CB2
 P 3350 950
-F 0 "TH?" H 3100 1050 50  0000 C CNN
+F 0 "TH2" H 3100 1050 50  0000 C CNN
 F 1 "10k / 1% / 3454K / SMD0603" H 2550 950 50  0000 C CNN
-F 2 "" H 3350 1000 50  0001 C CNN
+F 2 "Resistors_SMD:R_0603" H 3350 1000 50  0001 C CNN
 F 3 "" H 3350 1000 50  0001 C CNN
 	1    3350 950
@@
 	3800 1600 4300 1600
 Wire Wire Line
-	3800 1100 3800 1500
-Wire Wire Line
-	3800 1500 3800 1600
-Wire Wire Line
-	3700 1500 3800 1500
-Wire Wire Line
-	3800 1500 3850 1500
+	3800 1100 3800 1600
+Wire Wire Line
+	3700 1500 3850 1500
 Connection ~ 3800 1500
 Wire Wire Line
@@
 5V_3
 Wire Wire Line
-	2750 650  3350 650
-Wire Wire Line
-	3350 650  3800 650
+	2750 650  3800 650
 Wire Wire Line
 	3350 650  3350 800
@@
 Connection ~ 3350 650
 $Comp
-L R R?
+L R R113
 U 1 1 592E4864
 P 2650 3700
-F 0 "R?" V 2750 3700 50  0000 C CNN
+F 0 "R113" V 2750 3700 50  0000 C CNN
 F 1 "1.82k / 0.063W / 1% / SMD 0603" V 2850 4200 50  0000 C CNN
-F 2 "" V 2580 3700 50  0001 C CNN
+F 2 "Resistors_SMD:R_0603" V 2580 3700 50  0001 C CNN
 F 3 "" H 2650 3700 50  0001 C CNN
 	1    2650 3700
@@
 $EndComp
 $Comp
-L R R?
+L R R112
 U 1 1 592E4932
 P 2100 3700
-F 0 "R?" V 2000 3700 50  0000 C CNN
+F 0 "R112" V 2000 3700 50  0000 C CNN
 F 1 "1.47k / 0.063W / 1% / SMD 0603" V 1900 3150 50  0000 C CNN
-F 2 "" V 2030 3700 50  0001 C CNN
+F 2 "Resistors_SMD:R_0603" V 2030 3700 50  0001 C CNN
 F 3 "" H 2100 3700 50  0001 C CNN
 	1    2100 3700
@@
 5V_3
 $Comp
-L C C?
+L C C58
 U 1 1 592E4B52
 P 2350 4100
-F 0 "C?" H 2375 4200 50  0000 L CNN
+F 0 "C58" H 2375 4200 50  0000 L CNN
 F 1 ".047 uF / 50V/ 10% / SMD 0603" H 2500 4100 50  0000 L CNN
 F 2 "Capacitors_SMD:C_0603" H 2388 3950 50  0001 C CNN
@@
 $EndComp
 $Comp
-L Thermistor_NTC TH?
+L Thermistor_NTC TH1
 U 1 1 592E4BBD
 P 1800 4100
-F 0 "TH?" H 1550 4200 50  0000 C CNN
+F 0 "TH1" H 1550 4200 50  0000 C CNN
 F 1 "10k / 1% / 3454K / SMD0603" H 1100 4100 50  0000 C CNN
-F 2 "" H 1800 4150 50  0001 C CNN
+F 2 "Resistors_SMD:R_0603" H 1800 4150 50  0001 C CNN
 F 3 "" H 1800 4150 50  0001 C CNN
 	1    1800 4100
@@
 	4300 3600 2350 3600
 Wire Wire Line
-	2350 3600 2350 3700
-Wire Wire Line
-	2350 3700 2350 3950
-Wire Wire Line
-	2250 3700 2350 3700
-Wire Wire Line
-	2350 3700 2500 3700
+	2350 3600 2350 3950
+Wire Wire Line
+	2250 3700 2500 3700
 Connection ~ 2350 3700
 Wire Wire Line
@@
 	1800 3700 1950 3700
 Wire Wire Line
-	1650 4450 1800 4450
-Wire Wire Line
-	1800 4450 2350 4450
+	1650 4450 2350 4450
 Wire Wire Line
 	1800 4450 1800 4250

Commit message: more WIP
TODO:
Fix pin 50
ground planes
figure out GND_2 weirdness
fix optoisolator 3d model
bq IC 3d model
triple check everything
BOM
Parts:
- added C66: 3.3 nF / 50V/ 10% / SMD 0603, Capacitors_SMD:C_0603, symbol C
- added C67, C68, C69: 33 pF / 50V/ 10% / SMD 0603, Capacitors_SMD:C_0603, symbol C
Connections:
- net CS_S: now also C67.1
- net GND_3: now also C66.1, C67.2, C68.2, C69.2
- net SCLK_S: now also C69.1
- net SDI_S: now also C68.1
- new net GND_2: C66.2
Other:
- moved on the sheet: R110
Changed lines of the file:
@@
 Text HLabel 5900 5850 3    60   Input ~ 0
 SCLK_S
-Text HLabel 5950 7100 0    60   Input ~ 0
+Text HLabel 1900 6650 0    60   Input ~ 0
 VDDHV
-Text HLabel 5950 7350 0    60   Input ~ 0
+Text HLabel 1900 6850 0    60   Input ~ 0
 GND
-Text GLabel 6100 7100 2    60   Input ~ 0
+Text GLabel 2050 6650 2    60   Input ~ 0
 VDDHV_3
-Text GLabel 6100 7350 2    60   Input ~ 0
+Text GLabel 2050 6850 2    60   Input ~ 0
 GND_3
 $Comp
@@
 $EndComp
 Wire Wire Line
-	5950 7100 6100 7100
-Wire Wire Line
-	6100 7350 5950 7350
+	1900 6650 2050 6650
+Wire Wire Line
+	2050 6850 1900 6850
 Wire Wire Line
 	5900 4350 5900 5850
@@
 	6000 5000 6000 5850
 Wire Wire Line
-	5600 5850 5600 4350
+	5600 4350 5600 5850
 $Comp
 L C C43
@@
 L R R110
 U 1 1 592E769E
-P 4600 5050
-F 0 "R110" H 4350 4950 50  0000 C CNN
-F 1 "100K0 / 0.063W / 5% / SMD 0603" H 3800 5050 50  0000 C CNN
-F 2 "Resistors_SMD:R_0603" V 4530 5050 50  0001 C CNN
-F 3 "" H 4600 5050 50  0001 C CNN
-	1    4600 5050
-	1    0    0    -1
-$EndComp
-Wire Wire Line
-	4600 4350 4600 4900
+P 4600 4950
+F 0 "R110" H 4350 4850 50  0000 C CNN
+F 1 "100K0 / 0.063W / 5% / SMD 0603" H 3800 4950 50  0000 C CNN
+F 2 "Resistors_SMD:R_0603" V 4530 4950 50  0001 C CNN
+F 3 "" H 4600 4950 50  0001 C CNN
+	1    4600 4950
+	1    0    0    -1
+$EndComp
+Wire Wire Line
+	4600 4350 4600 4800
 Text GLabel 2300 2150 0    60   Input ~ 0
 LDOA_3
 Connection ~ 2500 2150
-Text GLabel 4600 5500 3    60   Input ~ 0
+Text GLabel 4600 5300 3    60   Input ~ 0
 LDOA_3
 Wire Wire Line
-	4600 5200 4600 5500
+	4600 5100 4600 5300
 $Comp
 L C C59
@@
 	2350 4450 2350 4250
 Connection ~ 1800 4450
+$Comp
+L C C68
+U 1 1 5945AE24
+P 5100 5200
+F 0 "C68" H 5125 5300 50  0000 L CNN
+F 1 "33 pF / 50V/ 10% / SMD 0603" V 5250 4000 50  0000 L CNN
+F 2 "Capacitors_SMD:C_0603" H 5138 5050 50  0001 C CNN
+F 3 "" H 5100 5200 50  0001 C CNN
+	1    5100 5200
+	1    0    0    -1
+$EndComp
+$Comp
+L C C67
+U 1 1 5945AEB2
+P 4800 4800
+F 0 "C67" H 4825 4900 50  0000 L CNN
+F 1 "33 pF / 50V/ 10% / SMD 0603" V 4950 3600 50  0000 L CNN
+F 2 "Capacitors_SMD:C_0603" H 4838 4650 50  0001 C CNN
+F 3 "" H 4800 4800 50  0001 C CNN
+	1    4800 4800
+	1    0    0    -1
+$EndComp
+$Comp
+L C C69
+U 1 1 5945AF26
+P 5400 5650
+F 0 "C69" H 5425 5750 50  0000 L CNN
+F 1 "33 pF / 50V/ 10% / SMD 0603" V 5500 4300 50  0000 L CNN
+F 2 "Capacitors_SMD:C_0603" H 5438 5500 50  0001 C CNN
+F 3 "" H 5400 5650 50  0001 C CNN
+	1    5400 5650
+	1    0    0    -1
+$EndComp
+Wire Wire Line
+	4800 4650 4800 4500
+Wire Wire Line
+	4800 4500 5600 4500
+Connection ~ 5600 4500
+Wire Wire Line
+	5100 5050 5100 4600
+Wire Wire Line
+	5100 4600 5700 4600
+Connection ~ 5700 4600
+Wire Wire Line
+	5400 5500 5400 4750
+Wire Wire Line
+	5400 4750 5900 4750
+Connection ~ 5900 4750
+Text GLabel 4800 5050 3    60   Input ~ 0
+GND_3
+Text GLabel 5100 5500 3    60   Input ~ 0
+GND_3
+Text GLabel 5400 5950 3    60   Input ~ 0
+GND_3
+Wire Wire Line
+	4800 4950 4800 5150
+Wire Wire Line
+	5100 5500 5100 5350
+Wire Wire Line
+	5400 5950 5400 5800
+Text GLabel 2050 7400 2    60   Input ~ 0
+GND_2
+$Comp
+L C C66
+U 1 1 59462CEE
+P 1950 7150
+F 0 "C66" H 1975 7250 50  0000 L CNN
+F 1 "3.3 nF / 50V/ 10% / SMD 0603" H 1975 7050 50  0000 L CNN
+F 2 "Capacitors_SMD:C_0603" H 1988 7000 50  0001 C CNN
+F 3 "" H 1950 7150 50  0001 C CNN
+	1    1950 7150
+	1    0    0    -1
+$EndComp
+Wire Wire Line
+	2050 7400 1950 7400
+Wire Wire Line
+	1950 7400 1950 7300
+Wire Wire Line
+	1950 7000 1950 6850
+Connection ~ 1950 6850
 $EndSCHEMATC
