File: RLOOP_BMS_V2/Batt Conn.sch (KiCad schematic (older format))
At the start: 1 part, among them J2 2-1586041-0

Commit message: footprint and layout work WIP
Parts:
- J2: footprint (none) -> rLoop_Footprints:TE_2-1586041-0-2x10
Changed lines of the file:
@@
 F 0 "J2" H 5150 4400 50  0000 C CNN
 F 1 "2-1586041-0" V 5150 3850 50  0000 C CNN
-F 2 "" H 5150 2650 50  0001 C CNN
+F 2 "rLoop_Footprints:TE_2-1586041-0-2x10" H 5150 2650 50  0001 C CNN
 F 3 "" H 5150 2650 50  0001 C CNN
 	1    5150 3850

Commit message: board layout wip
Parts:
- removed J2: 2-1586041-0, rLoop_Footprints:TE_2-1586041-0-2x10, symbol CONN_02X10
- added J2: 2-640387-0, rLoop_Footprints:TE_2-640387-0, symbol 2-640387-0
Other:
- note removed: "PINOUT NOT FINAL, MAY FLIP DURING LAYOUT"
Changed lines of the file:
@@
 Comment4 ""
 $EndDescr
-Text HLabel 4900 3400 0    60   Output ~ 0
+Text HLabel 5100 2700 0    60   Output ~ 0
 Cell_0
-Text HLabel 5400 3400 2    60   Output ~ 0
+Text HLabel 5100 2800 0    60   Output ~ 0
 Cell_1
-Text HLabel 4900 3500 0    60   Output ~ 0
+Text HLabel 5100 2900 0    60   Output ~ 0
 Cell_2
-Text HLabel 5400 3500 2    60   Output ~ 0
+Text HLabel 5100 3000 0    60   Output ~ 0
 Cell_3
-Text HLabel 4900 3600 0    60   Output ~ 0
+Text HLabel 5100 3100 0    60   Output ~ 0
 Cell_4
-Text HLabel 5400 3600 2    60   Output ~ 0
+Text HLabel 5100 3200 0    60   Output ~ 0
 Cell_5
-Text HLabel 4900 3700 0    60   Output ~ 0
+Text HLabel 5100 3300 0    60   Output ~ 0
 Cell_6
-Text HLabel 5400 3700 2    60   Output ~ 0
+Text HLabel 5100 3400 0    60   Output ~ 0
 Cell_7
-Text HLabel 4900 3800 0    60   Output ~ 0
+Text HLabel 5100 3500 0    60   Output ~ 0
 Cell_8
-Text HLabel 5400 3800 2    60   Output ~ 0
+Text HLabel 5100 3600 0    60   Output ~ 0
 Cell_9
-Text HLabel 4900 3900 0    60   Output ~ 0
+Text HLabel 5100 3700 0    60   Output ~ 0
 Cell_10
-Text HLabel 5400 3900 2    60   Output ~ 0
+Text HLabel 5100 3800 0    60   Output ~ 0
 Cell_11
-Text HLabel 4900 4000 0    60   Output ~ 0
+Text HLabel 5100 3900 0    60   Output ~ 0
 Cell_12
-Text HLabel 5400 4000 2    60   Output ~ 0
+Text HLabel 5100 4000 0    60   Output ~ 0
 Cell_13
-Text HLabel 4900 4100 0    60   Output ~ 0
+Text HLabel 5100 4100 0    60   Output ~ 0
 Cell_14
-Text HLabel 5400 4100 2    60   Output ~ 0
+Text HLabel 5100 4200 0    60   Output ~ 0
 Cell_15
-Text HLabel 4900 4200 0    60   Output ~ 0
+Text HLabel 5100 4300 0    60   Output ~ 0
 Cell_16
-Text HLabel 5400 4200 2    60   Output ~ 0
+Text HLabel 5100 4400 0    60   Output ~ 0
 Cell_17
-Text HLabel 4900 4300 0    60   Output ~ 0
+Text HLabel 5100 4500 0    60   Output ~ 0
 Cell_18
-Text Notes 4150 4500 0    60   ~ 12
-PINOUT NOT FINAL, MAY FLIP DURING LAYOUT
+Text Notes 4400 2450 0    60   ~ 12
+Cell 0 is the negative terminal of the battery pack.
 $Comp
-L CONN_02X10 J2
-U 1 1 59149FEF
-P 5150 3850
-F 0 "J2" H 5150 4400 50  0000 C CNN
-F 1 "2-1586041-0" V 5150 3850 50  0000 C CNN
-F 2 "rLoop_Footprints:TE_2-1586041-0-2x10" H 5150 2650 50  0001 C CNN
-F 3 "" H 5150 2650 50  0001 C CNN
-	1    5150 3850
-	1    0    0    -1
+L 2-640387-0 J2
+U 1 1 5919474D
+P 5300 3650
+F 0 "J2" V 5500 4000 60  0000 C CNN
+F 1 "2-640387-0" V 5500 3150 60  0000 C CNN
+F 2 "rLoop_Footprints:TE_2-640387-0" H 5200 3150 60  0001 C CNN
+F 3 "" H 5200 3150 60  0001 C CNN
+	1    5300 3650
+	1    0    0    1
 $EndComp
-Text Notes 4100 3150 0    60   ~ 12
-Cell 0 is the negative terminal of the battery pack.
-NoConn ~ 5400 4300
+NoConn ~ 5100 4600
 $EndSCHEMATC

Commit message: More PCB Work
Should be done, needs final check on the stencil and solder mask around
the ata6870 thermal pad
Parts:
- J2: Source (none) -> www.mouser.com/somethingeroher
Changed lines of the file:
@@
 F 2 "rLoop_Footprints:TE_2-640387-0" H 5200 3150 60  0001 C CNN
 F 3 "" H 5200 3150 60  0001 C CNN
+F 4 "www.mouser.com/somethingeroher" V 5300 3650 60  0001 C CNN "Source"
 	1    5300 3650
 	1    0    0    1
