File: POWER_NODE_V2/Power Input.sch (KiCad schematic (older format))
At the start: 10 parts, among them J1 TE_1744055-2, J2 TE_1744055-2, J3 Keystone_3544-2, J4 Keystone_3544-2

Commit message: Lot's of progress
Parts:
- D1, D2: footprint rLoop Footprints:LED_0805 -> rLoop_Footprints:LED_0805
- D3, D4: value AS4PM-M3/86A -> FES10G; footprint rLoop Footprints:TO-277A_SMPC -> rLoop_Footprints:TO-277A_SMPC
- J1, J2: value TE_1744055-2 -> TE_3-641119-2; footprint rLoop Footprints:TE_1744055-2_3.96_EP_HDR_ASSY_2P_VERT_HT -> rLoop_Footprints:3-641119-2_TE_2P_MTA156_HDR
- J3, J4: footprint rLoop Footprints:Keystone_3544-2 -> rLoop_Footprints:Keystone_3544-2
Changed lines of the file:
@@
 P 4400 2450
 F 0 "J1" H 4400 2600 50  0000 C CNN
-F 1 "TE_1744055-2" V 4500 2450 50  0000 C CNN
-F 2 "rLoop Footprints:TE_1744055-2_3.96_EP_HDR_ASSY_2P_VERT_HT" H 4400 2450 50  0001 C CNN
+F 1 "TE_3-641119-2" V 4500 2450 50  0000 C CNN
+F 2 "rLoop_Footprints:3-641119-2_TE_2P_MTA156_HDR" H 4400 2450 50  0001 C CNN
 F 3 "" H 4400 2450 50  0001 C CNN
 	1    4400 2450
@@
 F 0 "J3" H 5200 2350 50  0000 C CNN
 F 1 "Keystone_3544-2" V 5300 2200 50  0000 C CNN
-F 2 "rLoop Footprints:Keystone_3544-2" H 5200 2200 50  0001 C CNN
+F 2 "rLoop_Footprints:Keystone_3544-2" H 5200 2200 50  0001 C CNN
 F 3 "" H 5200 2200 50  0001 C CNN
 	1    5200 2200
@@
 P 6500 2400
 F 0 "D3" H 6500 2500 50  0000 C CNN
-F 1 "AS4PM-M3/86A" H 6500 2300 50  0000 C CNN
-F 2 "rLoop Footprints:TO-277A_SMPC" H 6500 2400 50  0001 C CNN
+F 1 "FES10G" H 6500 2300 50  0000 C CNN
+F 2 "rLoop_Footprints:TO-277A_SMPC" H 6500 2400 50  0001 C CNN
 F 3 "" H 6500 2400 50  0001 C CNN
 	1    6500 2400
@@
 P 4400 4150
 F 0 "J2" H 4400 4300 50  0000 C CNN
-F 1 "TE_1744055-2" V 4500 4150 50  0000 C CNN
-F 2 "rLoop Footprints:TE_1744055-2_3.96_EP_HDR_ASSY_2P_VERT_HT" H 4400 4150 50  0001 C CNN
+F 1 "TE_3-641119-2" V 4500 4150 50  0000 C CNN
+F 2 "rLoop_Footprints:3-641119-2_TE_2P_MTA156_HDR" H 4400 4150 50  0001 C CNN
 F 3 "" H 4400 4150 50  0001 C CNN
 	1    4400 4150
@@
 F 0 "J4" H 5200 4050 50  0000 C CNN
 F 1 "Keystone_3544-2" V 5300 3900 50  0000 C CNN
-F 2 "rLoop Footprints:Keystone_3544-2" H 5200 3900 50  0001 C CNN
+F 2 "rLoop_Footprints:Keystone_3544-2" H 5200 3900 50  0001 C CNN
 F 3 "" H 5200 3900 50  0001 C CNN
 	1    5200 3900
@@
 P 6500 4100
 F 0 "D4" H 6500 4200 50  0000 C CNN
-F 1 "AS4PM-M3/86A" H 6500 4000 50  0000 C CNN
-F 2 "rLoop Footprints:TO-277A_SMPC" H 6500 4100 50  0001 C CNN
+F 1 "FES10G" H 6500 4000 50  0000 C CNN
+F 2 "rLoop_Footprints:TO-277A_SMPC" H 6500 4100 50  0001 C CNN
 F 3 "" H 6500 4100 50  0001 C CNN
 	1    6500 4100
@@
 F 0 "D2" V 5900 4700 50  0000 C CNN
 F 1 "EL-17-21VGC/TR8" V 6000 4350 50  0000 C CNN
-F 2 "rLoop Footprints:LED_0805" H 5950 4850 50  0001 C CNN
+F 2 "rLoop_Footprints:LED_0805" H 5950 4850 50  0001 C CNN
 F 3 "" H 5950 4850 50  0001 C CNN
 	1    5950 4850
@@
 F 0 "D1" V 5900 3000 50  0000 C CNN
 F 1 "EL-17-21VGC/TR8" V 6000 2650 50  0000 C CNN
-F 2 "rLoop Footprints:LED_0805" H 5950 3150 50  0001 C CNN
+F 2 "rLoop_Footprints:LED_0805" H 5950 3150 50  0001 C CNN
 F 3 "" H 5950 3150 50  0001 C CNN
 	1    5950 3150

Commit message: Added tooling holes & fiducial marks
Parts:
- D1, D2: symbol LED -> LED-RESCUE-POWER_NODE_V2
Changed lines of the file:
@@
 EESchema Schematic File Version 2
+LIBS:POWER_NODE_V2-rescue
 LIBS:power
 LIBS:device
@@
 $Descr A4 11693 8268
 encoding utf-8
-Sheet 2 9
+Sheet 2 10
 Title ""
 Date ""
@@
 Connection ~ 5950 2400
 $Comp
-L GND #PWR01
+L GND #PWR3
 U 1 1 5952286D
 P 5950 3450
-F 0 "#PWR01" H 5950 3200 50  0001 C CNN
+F 0 "#PWR3" H 5950 3200 50  0001 C CNN
 F 1 "GND" H 5950 3300 50  0000 C CNN
 F 2 "" H 5950 3450 50  0001 C CNN
@@
 Connection ~ 5950 4100
 $Comp
-L GND #PWR02
+L GND #PWR4
 U 1 1 59522A7A
 P 5950 5150
-F 0 "#PWR02" H 5950 4900 50  0001 C CNN
+F 0 "#PWR4" H 5950 4900 50  0001 C CNN
 F 1 "GND" H 5950 5000 50  0000 C CNN
 F 2 "" H 5950 5150 50  0001 C CNN
@@
 	7850 4100 6650 4100
 $Comp
-L +24V #PWR03
+L +24V #PWR5
 U 1 1 59522AEA
 P 7850 2000
-F 0 "#PWR03" H 7850 1850 50  0001 C CNN
+F 0 "#PWR5" H 7850 1850 50  0001 C CNN
 F 1 "+24V" H 7850 2140 50  0000 C CNN
 F 2 "" H 7850 2000 50  0001 C CNN
@@
 DC BUS B
 $Comp
-L GND #PWR04
+L GND #PWR1
 U 1 1 5952F227
 P 4800 2700
-F 0 "#PWR04" H 4800 2450 50  0001 C CNN
+F 0 "#PWR1" H 4800 2450 50  0001 C CNN
 F 1 "GND" H 4800 2550 50  0000 C CNN
 F 2 "" H 4800 2700 50  0001 C CNN
@@
 	4800 2500 4600 2500
 $Comp
-L GND #PWR05
+L GND #PWR2
 U 1 1 5952F2BA
 P 4800 4350
-F 0 "#PWR05" H 4800 4100 50  0001 C CNN
+F 0 "#PWR2" H 4800 4100 50  0001 C CNN
 F 1 "GND" H 4800 4200 50  0000 C CNN
 F 2 "" H 4800 4350 50  0001 C CNN
@@
 	4800 4200 4600 4200
 $Comp
-L LED D2
+L LED-RESCUE-POWER_NODE_V2 D2
 U 1 1 59522A60
 P 5950 4850
@@
 $EndComp
 $Comp
-L LED D1
+L LED-RESCUE-POWER_NODE_V2 D1
 U 1 1 59522073
 P 5950 3150
