File: POWER_NODE_V2/BMS Interface.sch (KiCad schematic (older format))
At the start: 11 parts, among them J10 5-534998-7, J9 TE_3-641119-2, U12 NCV8405ADTRKG, U13 MAX14850AEE+, U14 MAX14850AEE+

Commit message: added cooling solenoid to pcb
Parts:
- D6: footprint Diodes_THT:D_DO-201_P15.24mm_Horizontal -> rLoop_Footprints:D_DO-201_P15.24mm_Horizontal
Changed lines of the file:
@@
 $EndComp
 $Comp
-L GND #PWR108
+L GND #PWR096
 U 1 1 594CA92D
 P 8050 3350
-F 0 "#PWR108" H 8050 3100 50  0001 C CNN
+F 0 "#PWR096" H 8050 3100 50  0001 C CNN
 F 1 "GND" H 8050 3200 50  0000 C CNN
 F 2 "" H 8050 3350 50  0001 C CNN
@@
 $EndComp
 $Comp
-L +3.3V #PWR105
+L +3.3V #PWR097
 U 1 1 594CAB5E
 P 6300 3550
-F 0 "#PWR105" H 6300 3400 50  0001 C CNN
+F 0 "#PWR097" H 6300 3400 50  0001 C CNN
 F 1 "+3.3V" H 6300 3690 50  0000 C CNN
 F 2 "" H 6300 3550 50  0001 C CNN
@@
 $EndComp
 $Comp
-L +3.3V #PWR100
+L +3.3V #PWR098
 U 1 1 594CBADD
 P 4150 1350
-F 0 "#PWR100" H 4150 1200 50  0001 C CNN
+F 0 "#PWR098" H 4150 1200 50  0001 C CNN
 F 1 "+3.3V" H 4150 1490 50  0000 C CNN
 F 2 "" H 4150 1350 50  0001 C CNN
@@
 $EndComp
 $Comp
-L +3.3V #PWR98
+L +3.3V #PWR099
 U 1 1 594CBAF4
 P 2700 1350
-F 0 "#PWR98" H 2700 1200 50  0001 C CNN
+F 0 "#PWR099" H 2700 1200 50  0001 C CNN
 F 1 "+3.3V" H 2700 1490 50  0000 C CNN
 F 2 "" H 2700 1350 50  0001 C CNN
@@
 $EndComp
 $Comp
-L +3.3V #PWR102
+L +3.3V #PWR0100
 U 1 1 594CBB5B
 P 4150 3950
-F 0 "#PWR102" H 4150 3800 50  0001 C CNN
+F 0 "#PWR0100" H 4150 3800 50  0001 C CNN
 F 1 "+3.3V" H 4150 4090 50  0000 C CNN
 F 2 "" H 4150 3950 50  0001 C CNN
@@
 $EndComp
 $Comp
-L GND #PWR101
+L GND #PWR0101
 U 1 1 594CBF3C
 P 4150 3200
-F 0 "#PWR101" H 4150 2950 50  0001 C CNN
+F 0 "#PWR0101" H 4150 2950 50  0001 C CNN
 F 1 "GND" H 4150 3050 50  0000 C CNN
 F 2 "" H 4150 3200 50  0001 C CNN
@@
 $EndComp
 $Comp
-L GND #PWR103
+L GND #PWR0102
 U 1 1 594CBFA2
 P 4150 5800
-F 0 "#PWR103" H 4150 5550 50  0001 C CNN
+F 0 "#PWR0102" H 4150 5550 50  0001 C CNN
 F 1 "GND" H 4150 5650 50  0000 C CNN
 F 2 "" H 4150 5800 50  0001 C CNN
@@
 $EndComp
 $Comp
-L GND #PWR99
+L GND #PWR0103
 U 1 1 594DF3E0
 P 3750 7700
-F 0 "#PWR99" H 3750 7450 50  0001 C CNN
+F 0 "#PWR0103" H 3750 7450 50  0001 C CNN
 F 1 "GND" H 3750 7550 50  0000 C CNN
 F 2 "" H 3750 7700 50  0001 C CNN
@@
 $EndComp
 $Comp
-L +24V #PWR104
+L +24V #PWR0104
 U 1 1 594DF525
 P 4700 6300
-F 0 "#PWR104" H 4700 6150 50  0001 C CNN
+F 0 "#PWR0104" H 4700 6150 50  0001 C CNN
 F 1 "+24V" H 4700 6440 50  0000 C CNN
 F 2 "" H 4700 6300 50  0001 C CNN
@@
 $EndComp
 $Comp
-L +3.3V #PWR106
+L +3.3V #PWR0105
 U 1 1 59514C06
 P 6450 1550
-F 0 "#PWR106" H 6450 1400 50  0001 C CNN
+F 0 "#PWR0105" H 6450 1400 50  0001 C CNN
 F 1 "+3.3V" H 6450 1690 50  0000 C CNN
 F 2 "" H 6450 1550 50  0001 C CNN
@@
 $EndComp
 $Comp
-L +3.3V #PWR96
+L +3.3V #PWR0106
 U 1 1 5951542C
 P 2300 3850
-F 0 "#PWR96" H 2300 3700 50  0001 C CNN
+F 0 "#PWR0106" H 2300 3700 50  0001 C CNN
 F 1 "+3.3V" H 2300 3990 50  0000 C CNN
 F 2 "" H 2300 3850 50  0001 C CNN
@@
 $EndComp
 $Comp
-L GND #PWR97
+L GND #PWR0107
 U 1 1 59515432
 P 2300 4250
-F 0 "#PWR97" H 2300 4000 50  0001 C CNN
+F 0 "#PWR0107" H 2300 4000 50  0001 C CNN
 F 1 "GND" H 2300 4100 50  0000 C CNN
 F 2 "" H 2300 4250 50  0001 C CNN
@@
 F 0 "D6" V 5250 6350 50  0000 C CNN
 F 1 "IN4004" V 5150 6400 50  0000 C CNN
-F 2 "Diodes_THT:D_DO-201_P15.24mm_Horizontal" H 5200 6600 50  0001 C CNN
+F 2 "rLoop_Footprints:D_DO-201_P15.24mm_Horizontal" H 5200 6600 50  0001 C CNN
 F 3 "" H 5200 6600 50  0001 C CNN
 	1    5200 6600
@@
 BMS Interface
 $Comp
-L GND #PWR107
+L GND #PWR0108
 U 1 1 59514D0B
 P 6450 1950
-F 0 "#PWR107" H 6450 1700 50  0001 C CNN
+F 0 "#PWR0108" H 6450 1700 50  0001 C CNN
 F 1 "GND" H 6450 1800 50  0000 C CNN
 F 2 "" H 6450 1950 50  0001 C CNN
