File: POWER_NODE_V2/Charger Interface.sch (KiCad schematic (older format))
At the start: 42 parts, among them J11 CONN_01X04, J12 CONN_01X04, J13 TE_3-641119-2, J14 TE_3-641119-2, J15 TE_3-641119-2, U15 TL783CKTTR, U16 TL783CKTTR, U17 AMC1100DWV, U18 AMC1100DWV, U19 NUD3124LT1G, U20 RTE24024

Commit message: Added tooling holes & fiducial marks
Parts:
- D8: symbol LED -> LED-RESCUE-POWER_NODE_V2
Connections:
- net at D8.1 (K): now also R32.1
Changed lines of the file:
@@
 EESchema Schematic File Version 2
+LIBS:POWER_NODE_V2-rescue
 LIBS:power
 LIBS:device
@@
 $Descr USLetter 11000 8500
 encoding utf-8
-Sheet 8 9
+Sheet 8 10
 Title ""
 Date ""
@@
 $EndComp
 $Comp
-L +5V #PWR0109
+L +5V #PWR119
 U 1 1 594DBA09
 P 4350 4850
-F 0 "#PWR0109" H 4350 4700 50  0001 C CNN
+F 0 "#PWR119" H 4350 4700 50  0001 C CNN
 F 1 "+5V" H 4350 4990 50  0000 C CNN
 F 2 "" H 4350 4850 50  0001 C CNN
@@
 $EndComp
 $Comp
-L GND #PWR0110
+L GND #PWR113
 U 1 1 594DBA49
 P 2700 5000
-F 0 "#PWR0110" H 2700 4750 50  0001 C CNN
+F 0 "#PWR113" H 2700 4750 50  0001 C CNN
 F 1 "GND" H 2700 4850 50  0000 C CNN
 F 2 "" H 2700 5000 50  0001 C CNN
@@
 $EndComp
 $Comp
-L GND #PWR0111
+L GND #PWR109
 U 1 1 594DBA8D
 P 1300 5000
-F 0 "#PWR0111" H 1300 4750 50  0001 C CNN
+F 0 "#PWR109" H 1300 4750 50  0001 C CNN
 F 1 "GND" H 1300 4850 50  0000 C CNN
 F 2 "" H 1300 5000 50  0001 C CNN
@@
 $EndComp
 $Comp
-L GND #PWR0112
+L GND #PWR110
 U 1 1 594DBAD4
 P 1300 5850
-F 0 "#PWR0112" H 1300 5600 50  0001 C CNN
+F 0 "#PWR110" H 1300 5600 50  0001 C CNN
 F 1 "GND" H 1300 5700 50  0000 C CNN
 F 2 "" H 1300 5850 50  0001 C CNN
@@
 $EndComp
 $Comp
-L GND #PWR0113
+L GND #PWR114
 U 1 1 594DBB1D
 P 2700 5850
-F 0 "#PWR0113" H 2700 5600 50  0001 C CNN
+F 0 "#PWR114" H 2700 5600 50  0001 C CNN
 F 1 "GND" H 2700 5700 50  0000 C CNN
 F 2 "" H 2700 5850 50  0001 C CNN
@@
 $EndComp
 $Comp
-L GND #PWR0114
+L GND #PWR117
 U 1 1 594DBB5D
 P 4200 4850
-F 0 "#PWR0114" H 4200 4600 50  0001 C CNN
+F 0 "#PWR117" H 4200 4600 50  0001 C CNN
 F 1 "GND" H 4200 4700 50  0000 C CNN
 F 2 "" H 4200 4850 50  0001 C CNN
@@
 $EndComp
 $Comp
-L +5V #PWR0115
+L +5V #PWR120
 U 1 1 594DBD39
 P 4350 6700
-F 0 "#PWR0115" H 4350 6550 50  0001 C CNN
+F 0 "#PWR120" H 4350 6550 50  0001 C CNN
 F 1 "+5V" H 4350 6840 50  0000 C CNN
 F 2 "" H 4350 6700 50  0001 C CNN
@@
 $EndComp
 $Comp
-L GND #PWR0116
+L GND #PWR115
 U 1 1 594DBD41
 P 2700 6800
-F 0 "#PWR0116" H 2700 6550 50  0001 C CNN
+F 0 "#PWR115" H 2700 6550 50  0001 C CNN
 F 1 "GND" H 2700 6650 50  0000 C CNN
 F 2 "" H 2700 6800 50  0001 C CNN
@@
 $EndComp
 $Comp
-L GND #PWR0117
+L GND #PWR111
 U 1 1 594DBD48
 P 1300 6800
-F 0 "#PWR0117" H 1300 6550 50  0001 C CNN
+F 0 "#PWR111" H 1300 6550 50  0001 C CNN
 F 1 "GND" H 1300 6650 50  0000 C CNN
 F 2 "" H 1300 6800 50  0001 C CNN
@@
 $EndComp
 $Comp
-L GND #PWR0118
+L GND #PWR112
 U 1 1 594DBD4F
 P 1300 7650
-F 0 "#PWR0118" H 1300 7400 50  0001 C CNN
+F 0 "#PWR112" H 1300 7400 50  0001 C CNN
 F 1 "GND" H 1300 7500 50  0000 C CNN
 F 2 "" H 1300 7650 50  0001 C CNN
@@
 $EndComp
 $Comp
-L GND #PWR0119
+L GND #PWR116
 U 1 1 594DBD56
 P 2700 7650
-F 0 "#PWR0119" H 2700 7400 50  0001 C CNN
+F 0 "#PWR116" H 2700 7400 50  0001 C CNN
 F 1 "GND" H 2700 7500 50  0000 C CNN
 F 2 "" H 2700 7650 50  0001 C CNN
@@
 $EndComp
 $Comp
-L GND #PWR0120
+L GND #PWR118
 U 1 1 594DBD5D
 P 4200 6700
-F 0 "#PWR0120" H 4200 6450 50  0001 C CNN
+F 0 "#PWR118" H 4200 6450 50  0001 C CNN
 F 1 "GND" H 4200 6550 50  0000 C CNN
 F 2 "" H 4200 6700 50  0001 C CNN
@@
 $EndComp
 $Comp
-L GND #PWR0121
+L GND #PWR125
 U 1 1 594FF9E3
 P 6400 6300
-F 0 "#PWR0121" H 6400 6050 50  0001 C CNN
+F 0 "#PWR125" H 6400 6050 50  0001 C CNN
 F 1 "GND" H 6400 6150 50  0000 C CNN
 F 2 "" H 6400 6300 50  0001 C CNN
@@
 $EndComp
 $Comp
-L +24V #PWR0122
+L +24V #PWR129
 U 1 1 5950020D
 P 7850 4700
-F 0 "#PWR0122" H 7850 4550 50  0001 C CNN
+F 0 "#PWR129" H 7850 4550 50  0001 C CNN
 F 1 "+24V" H 7850 4840 50  0000 C CNN
 F 2 "" H 7850 4700 50  0001 C CNN
@@
 $EndComp
 $Comp
-L +24V #PWR0123
+L +24V #PWR128
 U 1 1 59500312
 P 7250 4700
-F 0 "#PWR0123" H 7250 4550 50  0001 C CNN
+F 0 "#PWR128" H 7250 4550 50  0001 C CNN
 F 1 "+24V" H 7250 4840 50  0000 C CNN
 F 2 "" H 7250 4700 50  0001 C CNN
@@
 $EndComp
 $Comp
-L GND #PWR0124
+L GND #PWR131
 U 1 1 595004C9
 P 9200 5600
-F 0 "#PWR0124" H 9200 5350 50  0001 C CNN
+F 0 "#PWR131" H 9200 5350 50  0001 C CNN
 F 1 "GND" H 9200 5450 50  0000 C CNN
 F 2 "" H 9200 5600 50  0001 C CNN
@@
 $EndComp
 $Comp
-L GND #PWR0125
+L GND #PWR130
 U 1 1 59500D07
 P 8950 6150
-F 0 "#PWR0125" H 8950 5900 50  0001 C CNN
+F 0 "#PWR130" H 8950 5900 50  0001 C CNN
 F 1 "GND" H 8950 6000 50  0000 C CNN
 F 2 "" H 8950 6150 50  0001 C CNN
@@
 $EndComp
 $Comp
-L +3V3 #PWR0126
+L +3V3 #PWR124
 U 1 1 5950349C
 P 6100 850
-F 0 "#PWR0126" H 6100 700 50  0001 C CNN
+F 0 "#PWR124" H 6100 700 50  0001 C CNN
 F 1 "+3V3" H 6100 990 50  0000 C CNN
 F 2 "" H 6100 850 50  0001 C CNN
@@
 $EndComp
 $Comp
-L GND #PWR0127
+L GND #PWR122
 U 1 1 5950366C
 P 6000 1950
-F 0 "#PWR0127" H 6000 1700 50  0001 C CNN
+F 0 "#PWR122" H 6000 1700 50  0001 C CNN
 F 1 "GND" H 6000 1800 50  0000 C CNN
 F 2 "" H 6000 1950 50  0001 C CNN
@@
 $EndComp
 $Comp
-L +3V3 #PWR0128
+L +3V3 #PWR123
 U 1 1 59505430
 P 6050 2450
-F 0 "#PWR0128" H 6050 2300 50  0001 C CNN
+F 0 "#PWR123" H 6050 2300 50  0001 C CNN
 F 1 "+3V3" H 6050 2590 50  0000 C CNN
 F 2 "" H 6050 2450 50  0001 C CNN
@@
 CHARGE_N_HOT
 $Comp
-L GND #PWR0129
+L GND #PWR127
 U 1 1 59515118
 P 7050 2550
-F 0 "#PWR0129" H 7050 2300 50  0001 C CNN
+F 0 "#PWR127" H 7050 2300 50  0001 C CNN
 F 1 "GND" H 7200 2500 50  0000 C CNN
 F 2 "" H 7050 2550 50  0001 C CNN
@@
 $EndComp
 $Comp
-L GND #PWR0130
+L GND #PWR126
 U 1 1 59515F53
 P 7050 900
-F 0 "#PWR0130" H 7050 650 50  0001 C CNN
+F 0 "#PWR126" H 7050 650 50  0001 C CNN
 F 1 "GND" H 7200 850 50  0000 C CNN
 F 2 "" H 7050 900 50  0001 C CNN
@@
 $EndComp
 $Comp
-L GND #PWR0131
+L GND #PWR121
 U 1 1 595056D5
 P 5950 3600
-F 0 "#PWR0131" H 5950 3350 50  0001 C CNN
+F 0 "#PWR121" H 5950 3350 50  0001 C CNN
 F 1 "GND" H 5950 3450 50  0000 C CNN
 F 2 "" H 5950 3600 50  0001 C CNN
@@
 Connection ~ 6950 5700
 $Comp
-L LED D8
+L LED-RESCUE-POWER_NODE_V2 D8
 U 1 1 5950058E
 P 8950 4900

Commit message: added cooling solenoid to pcb
Parts:
- D9: footprint Diodes_THT:D_DO-201_P15.24mm_Horizontal -> rLoop_Footprints:D_DO-201_P15.24mm_Horizontal
- U15, U16: footprint TO_SOT_Packages_SMD:TO-263-3_TabPin4 -> rLoop_Footprints:tl783ckttr
Changed lines of the file:
@@
 $EndComp
 $Comp
-L +5V #PWR119
+L +5V #PWR0109
 U 1 1 594DBA09
 P 4350 4850
-F 0 "#PWR119" H 4350 4700 50  0001 C CNN
+F 0 "#PWR0109" H 4350 4700 50  0001 C CNN
 F 1 "+5V" H 4350 4990 50  0000 C CNN
 F 2 "" H 4350 4850 50  0001 C CNN
@@
 $EndComp
 $Comp
-L GND #PWR113
+L GND #PWR0110
 U 1 1 594DBA49
 P 2700 5000
-F 0 "#PWR113" H 2700 4750 50  0001 C CNN
+F 0 "#PWR0110" H 2700 4750 50  0001 C CNN
 F 1 "GND" H 2700 4850 50  0000 C CNN
 F 2 "" H 2700 5000 50  0001 C CNN
@@
 $EndComp
 $Comp
-L GND #PWR109
+L GND #PWR0111
 U 1 1 594DBA8D
 P 1300 5000
-F 0 "#PWR109" H 1300 4750 50  0001 C CNN
+F 0 "#PWR0111" H 1300 4750 50  0001 C CNN
 F 1 "GND" H 1300 4850 50  0000 C CNN
 F 2 "" H 1300 5000 50  0001 C CNN
@@
 $EndComp
 $Comp
-L GND #PWR110
+L GND #PWR0112
 U 1 1 594DBAD4
 P 1300 5850
-F 0 "#PWR110" H 1300 5600 50  0001 C CNN
+F 0 "#PWR0112" H 1300 5600 50  0001 C CNN
 F 1 "GND" H 1300 5700 50  0000 C CNN
 F 2 "" H 1300 5850 50  0001 C CNN
@@
 $EndComp
 $Comp
-L GND #PWR114
+L GND #PWR0113
 U 1 1 594DBB1D
 P 2700 5850
-F 0 "#PWR114" H 2700 5600 50  0001 C CNN
+F 0 "#PWR0113" H 2700 5600 50  0001 C CNN
 F 1 "GND" H 2700 5700 50  0000 C CNN
 F 2 "" H 2700 5850 50  0001 C CNN
@@
 $EndComp
 $Comp
-L GND #PWR117
+L GND #PWR0114
 U 1 1 594DBB5D
 P 4200 4850
-F 0 "#PWR117" H 4200 4600 50  0001 C CNN
+F 0 "#PWR0114" H 4200 4600 50  0001 C CNN
 F 1 "GND" H 4200 4700 50  0000 C CNN
 F 2 "" H 4200 4850 50  0001 C CNN
@@
 $EndComp
 $Comp
-L +5V #PWR120
+L +5V #PWR0115
 U 1 1 594DBD39
 P 4350 6700
-F 0 "#PWR120" H 4350 6550 50  0001 C CNN
+F 0 "#PWR0115" H 4350 6550 50  0001 C CNN
 F 1 "+5V" H 4350 6840 50  0000 C CNN
 F 2 "" H 4350 6700 50  0001 C CNN
@@
 $EndComp
 $Comp
-L GND #PWR115
+L GND #PWR0116
 U 1 1 594DBD41
 P 2700 6800
-F 0 "#PWR115" H 2700 6550 50  0001 C CNN
+F 0 "#PWR0116" H 2700 6550 50  0001 C CNN
 F 1 "GND" H 2700 6650 50  0000 C CNN
 F 2 "" H 2700 6800 50  0001 C CNN
@@
 $EndComp
 $Comp
-L GND #PWR111
+L GND #PWR0117
 U 1 1 594DBD48
 P 1300 6800
-F 0 "#PWR111" H 1300 6550 50  0001 C CNN
+F 0 "#PWR0117" H 1300 6550 50  0001 C CNN
 F 1 "GND" H 1300 6650 50  0000 C CNN
 F 2 "" H 1300 6800 50  0001 C CNN
@@
 $EndComp
 $Comp
-L GND #PWR112
+L GND #PWR0118
 U 1 1 594DBD4F
 P 1300 7650
-F 0 "#PWR112" H 1300 7400 50  0001 C CNN
+F 0 "#PWR0118" H 1300 7400 50  0001 C CNN
 F 1 "GND" H 1300 7500 50  0000 C CNN
 F 2 "" H 1300 7650 50  0001 C CNN
@@
 $EndComp
 $Comp
-L GND #PWR116
+L GND #PWR0119
 U 1 1 594DBD56
 P 2700 7650
-F 0 "#PWR116" H 2700 7400 50  0001 C CNN
+F 0 "#PWR0119" H 2700 7400 50  0001 C CNN
 F 1 "GND" H 2700 7500 50  0000 C CNN
 F 2 "" H 2700 7650 50  0001 C CNN
@@
 $EndComp
 $Comp
-L GND #PWR118
+L GND #PWR0120
 U 1 1 594DBD5D
 P 4200 6700
-F 0 "#PWR118" H 4200 6450 50  0001 C CNN
+F 0 "#PWR0120" H 4200 6450 50  0001 C CNN
 F 1 "GND" H 4200 6550 50  0000 C CNN
 F 2 "" H 4200 6700 50  0001 C CNN
@@
 $EndComp
 $Comp
-L GND #PWR125
+L GND #PWR0121
 U 1 1 594FF9E3
 P 6400 6300
-F 0 "#PWR125" H 6400 6050 50  0001 C CNN
+F 0 "#PWR0121" H 6400 6050 50  0001 C CNN
 F 1 "GND" H 6400 6150 50  0000 C CNN
 F 2 "" H 6400 6300 50  0001 C CNN
@@
 F 0 "D9" V 9250 5150 50  0000 C CNN
 F 1 "1N4004" V 9150 5250 50  0000 C CNN
-F 2 "Diodes_THT:D_DO-201_P15.24mm_Horizontal" H 9200 5000 50  0001 C CNN
+F 2 "rLoop_Footprints:D_DO-201_P15.24mm_Horizontal" H 9200 5000 50  0001 C CNN
 F 3 "" H 9200 5000 50  0001 C CNN
 	1    9200 5000
@@
 $EndComp
 $Comp
-L +24V #PWR129
+L +24V #PWR0122
 U 1 1 5950020D
 P 7850 4700
-F 0 "#PWR129" H 7850 4550 50  0001 C CNN
+F 0 "#PWR0122" H 7850 4550 50  0001 C CNN
 F 1 "+24V" H 7850 4840 50  0000 C CNN
 F 2 "" H 7850 4700 50  0001 C CNN
@@
 $EndComp
 $Comp
-L +24V #PWR128
+L +24V #PWR0123
 U 1 1 59500312
 P 7250 4700
-F 0 "#PWR128" H 7250 4550 50  0001 C CNN
+F 0 "#PWR0123" H 7250 4550 50  0001 C CNN
 F 1 "+24V" H 7250 4840 50  0000 C CNN
 F 2 "" H 7250 4700 50  0001 C CNN
@@
 $EndComp
 $Comp
-L GND #PWR131
+L GND #PWR0124
 U 1 1 595004C9
 P 9200 5600
-F 0 "#PWR131" H 9200 5350 50  0001 C CNN
+F 0 "#PWR0124" H 9200 5350 50  0001 C CNN
 F 1 "GND" H 9200 5450 50  0000 C CNN
 F 2 "" H 9200 5600 50  0001 C CNN
@@
 $EndComp
 $Comp
-L GND #PWR130
+L GND #PWR0125
 U 1 1 59500D07
 P 8950 6150
-F 0 "#PWR130" H 8950 5900 50  0001 C CNN
+F 0 "#PWR0125" H 8950 5900 50  0001 C CNN
 F 1 "GND" H 8950 6000 50  0000 C CNN
 F 2 "" H 8950 6150 50  0001 C CNN
@@
 F 0 "U15" H 2050 1400 60  0000 C CNN
 F 1 "TL783CKTTR" H 2250 1500 60  0000 C CNN
-F 2 "TO_SOT_Packages_SMD:TO-263-3_TabPin4" H 2300 1150 60  0001 C CNN
+F 2 "rLoop_Footprints:tl783ckttr" H 2300 1150 60  0001 C CNN
 F 3 "" H 2300 1150 60  0001 C CNN
 	1    2300 1150
@@
 F 0 "U16" H 2050 3050 60  0000 C CNN
 F 1 "TL783CKTTR" H 2250 3150 60  0000 C CNN
-F 2 "TO_SOT_Packages_SMD:TO-263-3_TabPin4" H 2300 2800 60  0001 C CNN
+F 2 "rLoop_Footprints:tl783ckttr" H 2300 2800 60  0001 C CNN
 F 3 "" H 2300 2800 60  0001 C CNN
 	1    2300 2800
@@
 $EndComp
 $Comp
-L +3V3 #PWR124
+L +3V3 #PWR0126
 U 1 1 5950349C
 P 6100 850
-F 0 "#PWR124" H 6100 700 50  0001 C CNN
+F 0 "#PWR0126" H 6100 700 50  0001 C CNN
 F 1 "+3V3" H 6100 990 50  0000 C CNN
 F 2 "" H 6100 850 50  0001 C CNN
@@
 $EndComp
 $Comp
-L GND #PWR122
+L GND #PWR0127
 U 1 1 5950366C
 P 6000 1950
-F 0 "#PWR122" H 6000 1700 50  0001 C CNN
+F 0 "#PWR0127" H 6000 1700 50  0001 C CNN
 F 1 "GND" H 6000 1800 50  0000 C CNN
 F 2 "" H 6000 1950 50  0001 C CNN
@@
 $EndComp
 $Comp
-L +3V3 #PWR123
+L +3V3 #PWR0128
 U 1 1 59505430
 P 6050 2450
-F 0 "#PWR123" H 6050 2300 50  0001 C CNN
+F 0 "#PWR0128" H 6050 2300 50  0001 C CNN
 F 1 "+3V3" H 6050 2590 50  0000 C CNN
 F 2 "" H 6050 2450 50  0001 C CNN
@@
 CHARGE_N_HOT
 $Comp
-L GND #PWR127
+L GND #PWR0129
 U 1 1 59515118
 P 7050 2550
-F 0 "#PWR127" H 7050 2300 50  0001 C CNN
+F 0 "#PWR0129" H 7050 2300 50  0001 C CNN
 F 1 "GND" H 7200 2500 50  0000 C CNN
 F 2 "" H 7050 2550 50  0001 C CNN
@@
 $EndComp
 $Comp
-L GND #PWR126
+L GND #PWR0130
 U 1 1 59515F53
 P 7050 900
-F 0 "#PWR126" H 7050 650 50  0001 C CNN
+F 0 "#PWR0130" H 7050 650 50  0001 C CNN
 F 1 "GND" H 7200 850 50  0000 C CNN
 F 2 "" H 7050 900 50  0001 C CNN
@@
 $EndComp
 $Comp
-L GND #PWR121
+L GND #PWR0131
 U 1 1 595056D5
 P 5950 3600
-F 0 "#PWR121" H 5950 3350 50  0001 C CNN
+F 0 "#PWR0131" H 5950 3350 50  0001 C CNN
 F 1 "GND" H 5950 3450 50  0000 C CNN
 F 2 "" H 5950 3600 50  0001 C CNN
