File: POWER_NODE_V2/Cooling Solenoid.sch (KiCad schematic (older format))
At the start: 8 parts, among them P1 TE_3-641119-2, U21 NUD3124LT1G, U22 RTE24024

Commit message: added cooling solenoid to pcb
Parts:
- D15: footprint Diodes_THT:D_DO-201_P15.24mm_Horizontal -> rLoop_Footprints:1N4004
Changed lines of the file:
@@
 F 0 "D15" V 8350 3100 50  0000 C CNN
 F 1 "1N4004" V 8250 3150 50  0000 C CNN
-F 2 "Diodes_THT:D_DO-201_P15.24mm_Horizontal" H 8300 3350 50  0001 C CNN
+F 2 "rLoop_Footprints:1N4004" H 8300 3350 50  0001 C CNN
 F 3 "" H 8300 3350 50  0000 C CNN
 	1    8300 3350
@@
 $EndComp
 $Comp
-L GND #PWR144
+L GND #PWR0144
 U 1 1 5965CD75
 P 4000 4700
-F 0 "#PWR144" H 4000 4450 50  0001 C CNN
+F 0 "#PWR0144" H 4000 4450 50  0001 C CNN
 F 1 "GND" H 4000 4550 50  0000 C CNN
 F 2 "" H 4000 4700 50  0000 C CNN
@@
 $EndComp
 $Comp
-L +24V #PWR146
+L +24V #PWR0145
 U 1 1 5965CE8C
 P 6100 3000
-F 0 "#PWR146" H 6100 2850 50  0001 C CNN
+F 0 "#PWR0145" H 6100 2850 50  0001 C CNN
 F 1 "+24V" H 6100 3140 50  0000 C CNN
 F 2 "" H 6100 3000 50  0000 C CNN
@@
 	8300 3500 8300 4350
 $Comp
-L GND #PWR148
+L GND #PWR0146
 U 1 1 5965D1A8
 P 8300 4350
-F 0 "#PWR148" H 8300 4100 50  0001 C CNN
+F 0 "#PWR0146" H 8300 4100 50  0001 C CNN
 F 1 "GND" H 8300 4200 50  0000 C CNN
 F 2 "" H 8300 4350 50  0000 C CNN
@@
 	7650 3900 7650 3550
 $Comp
-L GND #PWR147
+L GND #PWR0147
 U 1 1 5965D2D8
 P 7650 4350
-F 0 "#PWR147" H 7650 4100 50  0001 C CNN
+F 0 "#PWR0147" H 7650 4100 50  0001 C CNN
 F 1 "GND" H 7650 4200 50  0000 C CNN
 F 2 "" H 7650 4350 50  0000 C CNN
@@
 	4800 3250 5500 3250
 $Comp
-L +24V #PWR145
+L +24V #PWR0148
 U 1 1 5965D351
 P 5500 3000
-F 0 "#PWR145" H 5500 2850 50  0001 C CNN
+F 0 "#PWR0148" H 5500 2850 50  0001 C CNN
 F 1 "+24V" H 5500 3140 50  0000 C CNN
 F 2 "" H 5500 3000 50  0000 C CNN
